File: Hardware/Control_PCB/KiCAD_Project/control_pcb/Power.sch (KiCad schematic (older format))
At the start: 10 parts, among them J6 Battery, J7 External Switch, U7 LT1521-3.3

Commit message: Control PCB Rev 1.0 complete.
Parts:
- C16, C19: Internal Part Number 1-0000075 -> 1-0000005
Changed lines of the file:
@@
 F 2 "Capacitors_SMD:C_0603_HandSoldering" H 4888 3550 50  0001 C CNN
 F 3 "~" H 4850 3700 50  0001 C CNN
-F 4 "1-0000075" H 4850 3700 50  0001 C CNN "Internal Part Number"
+F 4 "1-0000005" H 4850 3700 50  0001 C CNN "Internal Part Number"
 F 5 "1" H 4850 3700 50  0001 C CNN "Populated"
 	1    4850 3700
@@
 F 2 "Capacitors_SMD:C_0603_HandSoldering" H 6888 3550 50  0001 C CNN
 F 3 "~" H 6850 3700 50  0001 C CNN
-F 4 "1-0000075" H 6850 3700 50  0001 C CNN "Internal Part Number"
+F 4 "1-0000005" H 6850 3700 50  0001 C CNN "Internal Part Number"
 F 5 "1" H 6850 3700 50  0001 C CNN "Populated"
 	1    6850 3700
