File: Hardware/Control_PCB/KiCAD_Project/control_pcb/Power.sch (KiCad schematic (older format))
At the start: 10 parts, among them J6 Battery, J7 External Switch, U7 LT1521-3.3

Commit message: Draft of next layout
Parts:
- removed C16, C19: 10u, Capacitors_SMD:C_0603_HandSoldering, symbol Device:C
- removed C17, C20: 1u, Capacitors_SMD:C_0603_HandSoldering, symbol Device:C
- removed C18, C21: 0.1u, Capacitors_SMD:C_0603_HandSoldering, symbol Device:C
- removed U7: LT1521-3.3, TO_SOT_Packages_SMD:SOT-223-3_TabPin2, symbol lib_sch:LT1521-3.3
- added C21, C22, C24, C25: 1-0000075, capacitors_0805:1-0000075, symbol capacitors_0805:1-0000075
- added C23, C26: 1-0000018, capacitors_0603:1-0000018, symbol capacitors_0603:1-0000018
- added D8: D_Schottky, Diode_SMD:D_SOD-123F, symbol Device:D_Schottky
- added R44, R45: 1-0000174, resistors_0603:1-0000174, symbol resistors_0603:1-0000174
- added U8, U9: SPX3819M5-L-3-3, Package_TO_SOT_SMD:SOT-23-5, symbol Regulator_Linear:SPX3819M5-L-3-3
- J8: renamed from J7; footprint Pin_Headers:Pin_Header_Straight_1x02_Pitch2.54mm -> Connector_PinHeader_2.54mm:PinHeader_1x02_P2.54mm_Vertical
- J9: renamed from J6; footprint Pin_Headers:Pin_Header_Straight_1x02_Pitch2.54mm -> Connector_PinHeader_2.54mm:PinHeader_1x02_P2.54mm_Vertical
Connections:
- net labels added: 3V3_XBEE
- wire segments 18 -> 31
- no-connect marks 0 -> 2
Other:
- note added: "Regulate the incoming voltage to the 3V3 needed for almost all components in the\ndesign. The fiber receiver/buffer uses raw battery voltage."
- moved on the sheet: F1, J8, J9

Commit message: Add final production files
Parts:
- D8: Internal Part Number (none) -> 1-0000669; Populated (none) -> 1
Changed lines of the file:
@@
 Sheet 6 6
 Title "Control Paddle Electronics - NSSL EFM"
-Date "2020-03-31"
-Rev "2.0"
+Date "2020-12-30"
+Rev "3.0"
 Comp "Leeman Geophysical LLC"
 Comment1 "(479) 373-3736"
@@
 	4500 3050 4700 3050
 $Comp
-L power:GND #PWR066
+L power:GND #PWR064
 U 1 1 5DF93731
 P 4175 3150
-F 0 "#PWR066" H 4175 2900 50  0001 C CNN
+F 0 "#PWR064" H 4175 2900 50  0001 C CNN
 F 1 "GND" H 4180 2977 50  0000 C CNN
 F 2 "" H 4175 3150 50  0001 C CNN
@@
 $EndComp
 $Comp
-L power:+BATT #PWR064
+L power:+BATT #PWR062
 U 1 1 5DF950EE
 P 5100 2850
-F 0 "#PWR064" H 5100 2700 50  0001 C CNN
+F 0 "#PWR062" H 5100 2700 50  0001 C CNN
 F 1 "+BATT" H 5115 3023 50  0000 C CNN
 F 2 "" H 5100 2850 50  0001 C CNN
@@
 	5100 3050 5000 3050
 $Comp
-L power:+3V3 #PWR065
+L power:+3V3 #PWR063
 U 1 1 5DF95B84
 P 7400 3050
-F 0 "#PWR065" H 7400 2900 50  0001 C CNN
+F 0 "#PWR063" H 7400 2900 50  0001 C CNN
 F 1 "+3V3" H 7415 3223 50  0000 C CNN
 F 2 "" H 7400 3050 50  0001 C CNN
@@
 $EndComp
 $Comp
-L power:GND #PWR070
+L power:GND #PWR068
 U 1 1 5FF8A980
 P 6475 3450
-F 0 "#PWR070" H 6475 3200 50  0001 C CNN
+F 0 "#PWR068" H 6475 3200 50  0001 C CNN
 F 1 "GND" H 6480 3277 50  0000 C CNN
 F 2 "" H 6475 3450 50  0001 C CNN
@@
 F 2 "Diode_SMD:D_SOD-123F" H 5325 3050 50  0001 C CNN
 F 3 "~" H 5325 3050 50  0001 C CNN
+F 4 "1-0000669" H 5325 3050 50  0001 C CNN "Internal Part Number"
+F 5 "1" H 5325 3050 50  0001 C CNN "Populated"
 	1    5325 3050
 	-1   0    0    1
@@
 $EndComp
 $Comp
-L power:GND #PWR067
+L power:GND #PWR065
 U 1 1 5FF8F68E
 P 5650 3375
-F 0 "#PWR067" H 5650 3125 50  0001 C CNN
+F 0 "#PWR065" H 5650 3125 50  0001 C CNN
 F 1 "GND" H 5655 3202 50  0000 C CNN
 F 2 "" H 5650 3375 50  0001 C CNN
@@
 Connection ~ 7250 3050
 $Comp
-L power:GND #PWR068
+L power:GND #PWR066
 U 1 1 5FF9243A
 P 7000 3375
-F 0 "#PWR068" H 7000 3125 50  0001 C CNN
+F 0 "#PWR066" H 7000 3125 50  0001 C CNN
 F 1 "GND" H 7005 3202 50  0000 C CNN
 F 2 "" H 7000 3375 50  0001 C CNN
@@
 $EndComp
 $Comp
-L power:GND #PWR069
+L power:GND #PWR067
 U 1 1 5FF92671
 P 7250 3375
-F 0 "#PWR069" H 7250 3125 50  0001 C CNN
+F 0 "#PWR067" H 7250 3125 50  0001 C CNN
 F 1 "GND" H 7255 3202 50  0000 C CNN
 F 2 "" H 7250 3375 50  0001 C CNN
@@
 $EndComp
 $Comp
-L power:GND #PWR026
+L power:GND #PWR069
 U 1 1 5FF1DFB5
 P 5650 4325
-F 0 "#PWR026" H 5650 4075 50  0001 C CNN
+F 0 "#PWR069" H 5650 4075 50  0001 C CNN
 F 1 "GND" H 5655 4152 50  0000 C CNN
 F 2 "" H 5650 4325 50  0001 C CNN
@@
 Connection ~ 7250 4000
 $Comp
-L power:GND #PWR029
+L power:GND #PWR070
 U 1 1 5FF1DFD8
 P 7000 4325
-F 0 "#PWR029" H 7000 4075 50  0001 C CNN
+F 0 "#PWR070" H 7000 4075 50  0001 C CNN
 F 1 "GND" H 7005 4152 50  0000 C CNN
 F 2 "" H 7000 4325 50  0001 C CNN

Commit message: Control Rev 3.1
Parts:
- removed R45: 1-0000174, resistors_0603:1-0000174, symbol resistors_0603:1-0000174
- removed U9: SPX3819M5-L-3-3, Package_TO_SOT_SMD:SOT-23-5, symbol Regulator_Linear:SPX3819M5-L-3-3
- added U9: 1-0000946, dc_dc_converters:1-0000946, symbol dc_dc_converters:1-0000946
Connections:
- net 3V3_XBEE: now also U9.6 (+Vout)
- net GND: now also U9.1 (GND), U9.7 (-Vout)
- net at C21.1, C24.1, D8.1 (K)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: now also U9.2 (Vcc)
Other:
- moved on the sheet: C25, C26
Changed lines of the file:
@@
 Sheet 6 6
 Title "Control Paddle Electronics - NSSL EFM"
-Date "2020-12-30"
-Rev "3.0"
+Date "2021-11-22"
+Rev "3.1"
 Comp "Leeman Geophysical LLC"
 Comment1 "(479) 373-3736"
@@
 Regulate the incoming voltage to the 3V3 needed for almost all components in the\ndesign. The fiber receiver/buffer uses raw battery voltage.
 Wire Wire Line
-	7250 4000 7400 4000
-$Comp
-L Regulator_Linear:SPX3819M5-L-3-3 U9
-U 1 1 5FF1DF92
-P 6475 4100
-F 0 "U9" H 6475 4442 50  0000 C CNN
-F 1 "SPX3819M5-L-3-3" H 6475 4351 50  0000 C CNN
-F 2 "Package_TO_SOT_SMD:SOT-23-5" H 6475 4425 50  0001 C CNN
-F 3 "https://www.exar.com/content/document.ashx?id=22106&languageid=1033&type=Datasheet&partnumber=SPX3819&filename=SPX3819.pdf&part=SPX3819" H 6475 4100 50  0001 C CNN
-F 4 "1-0000524" H 6475 4100 50  0001 C CNN "Internal Part Number"
-F 5 "1" H 6475 4100 50  0001 C CNN "Populated"
-	1    6475 4100
-	1    0    0    -1
-$EndComp
+	7600 4000 7750 4000
 $Comp
 L power:GND #PWR072
 U 1 1 5FF1DF98
-P 6475 4400
-F 0 "#PWR072" H 6475 4150 50  0001 C CNN
-F 1 "GND" H 6480 4227 50  0000 C CNN
-F 2 "" H 6475 4400 50  0001 C CNN
-F 3 "" H 6475 4400 50  0001 C CNN
-	1    6475 4400
+P 6925 4300
+F 0 "#PWR072" H 6925 4050 50  0001 C CNN
+F 1 "GND" H 6930 4127 50  0000 C CNN
+F 2 "" H 6925 4300 50  0001 C CNN
+F 3 "" H 6925 4300 50  0001 C CNN
+	1    6925 4300
 	1    0    0    -1
 $EndComp
-NoConn ~ 6775 4100
-$Comp
-L resistors_0603:1-0000174 R45
-U 1 1 5FF1DFA2
-P 5975 4175
-F 0 "R45" V 5900 4100 50  0000 L CNN
-F 1 "1-0000174" V 5975 4175 50  0001 C CNN
-F 2 "resistors_0603:1-0000174" V 5905 4175 50  0001 C CNN
-F 3 "~" H 5975 4175 50  0001 C CNN
-F 4 "1-0000174" H 5975 4175 50  0001 C CNN "Internal Part Number"
-F 5 "1" H 5975 4175 50  0001 C CNN "Populated"
-F 6 "100k" V 5975 4075 50  0000 L CNN "PValue"
-	1    5975 4175
-	1    0    0    -1
-$EndComp
-Wire Wire Line
-	5975 4325 6175 4325
-Wire Wire Line
-	6175 4325 6175 4100
-Wire Wire Line
-	5975 4025 5975 4000
-Wire Wire Line
-	5975 4000 6175 4000
 $Comp
 L capacitors_0805:1-0000075 C24
@@
 Wire Wire Line
 	5650 4000 5650 4025
-Wire Wire Line
-	5650 4000 5975 4000
-Connection ~ 5650 4000
-Connection ~ 5975 4000
 $Comp
 L capacitors_0805:1-0000075 C25
 U 1 1 5FF1DFC3
-P 7000 4175
-F 0 "C25" H 6750 4175 50  0000 L CNN
-F 1 "1-0000075" H 7025 4075 50  0001 L CNN
-F 2 "capacitors_0805:1-0000075" H 7038 4025 50  0001 C CNN
-F 3 "~" H 7000 4175 50  0001 C CNN
-F 4 "1-0000075" H 7000 4175 50  0001 C CNN "Internal Part Number"
-F 5 "1" H 7000 4175 50  0001 C CNN "Populated"
-F 6 "10uF" H 6725 4100 50  0000 L CNN "PValue"
-	1    7000 4175
+P 7350 4175
+F 0 "C25" H 7100 4175 50  0000 L CNN
+F 1 "1-0000075" H 7375 4075 50  0001 L CNN
+F 2 "capacitors_0805:1-0000075" H 7388 4025 50  0001 C CNN
+F 3 "~" H 7350 4175 50  0001 C CNN
+F 4 "1-0000075" H 7350 4175 50  0001 C CNN "Internal Part Number"
+F 5 "1" H 7350 4175 50  0001 C CNN "Populated"
+F 6 "10uF" H 7075 4100 50  0000 L CNN "PValue"
+	1    7350 4175
 	1    0    0    -1
 $EndComp
@@
 L capacitors_0603:1-0000018 C26
 U 1 1 5FF1DFCC
-P 7250 4175
-F 0 "C26" H 7350 4175 50  0000 L CNN
-F 1 "1-0000018" H 7275 4075 50  0001 L CNN
-F 2 "capacitors_0603:1-0000018" H 7288 4025 50  0001 C CNN
-F 3 "~" H 7250 4175 50  0001 C CNN
-F 4 "1-0000018" H 7250 4175 50  0001 C CNN "Internal Part Number"
-F 5 "1" H 7250 4175 50  0001 C CNN "Populated"
-F 6 "1uF" H 7350 4100 50  0000 L CNN "PValue"
-	1    7250 4175
+P 7600 4175
+F 0 "C26" H 7700 4175 50  0000 L CNN
+F 1 "1-0000018" H 7625 4075 50  0001 L CNN
+F 2 "capacitors_0603:1-0000018" H 7638 4025 50  0001 C CNN
+F 3 "~" H 7600 4175 50  0001 C CNN
+F 4 "1-0000018" H 7600 4175 50  0001 C CNN "Internal Part Number"
+F 5 "1" H 7600 4175 50  0001 C CNN "Populated"
+F 6 "1uF" H 7700 4100 50  0000 L CNN "PValue"
+	1    7600 4175
 	1    0    0    -1
 $EndComp
 Wire Wire Line
-	6775 4000 7000 4000
-Wire Wire Line
-	7000 4000 7000 4025
-Wire Wire Line
-	7000 4000 7250 4000
-Wire Wire Line
-	7250 4000 7250 4025
-Connection ~ 7000 4000
-Connection ~ 7250 4000
+	7350 4000 7350 4025
+Wire Wire Line
+	7350 4000 7600 4000
+Wire Wire Line
+	7600 4000 7600 4025
+Connection ~ 7600 4000
 $Comp
 L power:GND #PWR070
 U 1 1 5FF1DFD8
-P 7000 4325
-F 0 "#PWR070" H 7000 4075 50  0001 C CNN
-F 1 "GND" H 7005 4152 50  0000 C CNN
-F 2 "" H 7000 4325 50  0001 C CNN
-F 3 "" H 7000 4325 50  0001 C CNN
-	1    7000 4325
+P 7350 4325
+F 0 "#PWR070" H 7350 4075 50  0001 C CNN
+F 1 "GND" H 7355 4152 50  0000 C CNN
+F 2 "" H 7350 4325 50  0001 C CNN
+F 3 "" H 7350 4325 50  0001 C CNN
+	1    7350 4325
 	1    0    0    -1
 $EndComp
@@
 L power:GND #PWR071
 U 1 1 5FF1DFDE
-P 7250 4325
-F 0 "#PWR071" H 7250 4075 50  0001 C CNN
-F 1 "GND" H 7255 4152 50  0000 C CNN
-F 2 "" H 7250 4325 50  0001 C CNN
-F 3 "" H 7250 4325 50  0001 C CNN
-	1    7250 4325
+P 7600 4325
+F 0 "#PWR071" H 7600 4075 50  0001 C CNN
+F 1 "GND" H 7605 4152 50  0000 C CNN
+F 2 "" H 7600 4325 50  0001 C CNN
+F 3 "" H 7600 4325 50  0001 C CNN
+	1    7600 4325
 	1    0    0    -1
 $EndComp
@@
 Wire Wire Line
 	5500 4000 5650 4000
-Text GLabel 7400 4000 2    50   UnSpc ~ 0
+Text GLabel 7750 4000 2    50   UnSpc ~ 0
 3V3_XBEE
+Wire Wire Line
+	6025 4150 5850 4150
+Wire Wire Line
+	5850 4150 5850 4000
+Wire Wire Line
+	5850 4000 5650 4000
+Connection ~ 5650 4000
+$Comp
+L power:GND #PWR0101
+U 1 1 619AB9B3
+P 6025 4300
+F 0 "#PWR0101" H 6025 4050 50  0001 C CNN
+F 1 "GND" H 6030 4127 50  0000 C CNN
+F 2 "" H 6025 4300 50  0001 C CNN
+F 3 "" H 6025 4300 50  0001 C CNN
+	1    6025 4300
+	1    0    0    -1
+$EndComp
+NoConn ~ 6025 4000
+Wire Wire Line
+	6925 4000 7350 4000
+Connection ~ 7350 4000
+$Comp
+L dc_dc_converters:1-0000946 U?
+U 1 1 619A7A9B
+P 6475 4150
+AR Path="/619A7A9B" Ref="U?"  Part="1"
+AR Path="/5DF886D9/619A7A9B" Ref="U9"  Part="1"
+F 0 "U9" H 6750 4450 50  0000 C CNN
+F 1 "1-0000946" H 6475 4900 50  0001 C CNN
+F 2 "dc_dc_converters:1-0000946" H 6475 4550 50  0001 C CNN
+F 3 "" H 6475 4550 50  0001 C CNN
+F 4 "1-0000946" H 6475 4700 50  0001 C CNN "Internal Part Number"
+F 5 "1" H 6475 4800 50  0001 C CNN "Populated"
+F 6 "TMR 6" H 6475 3850 50  0000 C CNN "PValue"
+	1    6475 4150
+	1    0    0    -1
+$EndComp
 $EndSCHEMATC
