File: Hardware/Control_PCB/KiCAD_Project/control_pcb/control_pcb.sch (KiCad schematic (older format))
At the start: 34 parts, among them J1 Conn_01x02, J2 ISP, J3 Spare 2, SW1 Freq Select, U1 STM32F103CBT6, Y1 8MHz

Commit message: Change UARTS for separate radio serial.
Parts:
- J3: value Spare 2 -> Spare
Connections:
- net labels added: Unused_Fiber_Ser_TX, Unused_Radio_Ser_RX
- wire segments 103 -> 107
Other:
- moved on the sheet: R24, R25, R26, SW1
Changed lines of the file:
@@
 Text GLabel 5325 3425 0    50   Input ~ 0
 Radio_Serial_Select
-Text GLabel 6625 3425 2    50   Output ~ 0
+Text GLabel 5325 4025 0    50   Output ~ 0
 TX_to_Radio
 $Sheet
@@
 P 5000 3725
 F 0 "J3" H 5175 3725 50  0000 C CNN
-F 1 "Spare 2" H 5250 3600 50  0000 C CNN
+F 1 "Spare" H 5225 3650 50  0000 C CNN
 F 2 "Pin_Headers:Pin_Header_Straight_1x04_Pitch2.54mm" H 5000 3725 50  0001 C CNN
 F 3 "~" H 5000 3725 50  0001 C CNN
@@
 	-1   0    0    1
 $EndComp
-NoConn ~ 5325 4025
-NoConn ~ 5325 4125
 NoConn ~ 5325 4225
 NoConn ~ 5325 4325
@@
 L Device:R R24
 U 1 1 5DF76648
-P 4525 4325
-F 0 "R24" V 4600 4275 50  0000 L CNN
-F 1 "10k" V 4525 4250 50  0000 L CNN
-F 2 "Resistors_SMD:R_0603_HandSoldering" V 4455 4325 50  0001 C CNN
-F 3 "~" H 4525 4325 50  0001 C CNN
-F 4 "1-0000010" H 4525 4325 50  0001 C CNN "Internal Part Number"
-F 5 "1" H 4525 4325 50  0001 C CNN "Populated"
-	1    4525 4325
+P 3950 4325
+F 0 "R24" V 4025 4275 50  0000 L CNN
+F 1 "10k" V 3950 4250 50  0000 L CNN
+F 2 "Resistors_SMD:R_0603_HandSoldering" V 3880 4325 50  0001 C CNN
+F 3 "~" H 3950 4325 50  0001 C CNN
+F 4 "1-0000010" H 3950 4325 50  0001 C CNN "Internal Part Number"
+F 5 "1" H 3950 4325 50  0001 C CNN "Populated"
+	1    3950 4325
 	1    0    0    -1
 $EndComp
@@
 L Device:R R25
 U 1 1 5DF77109
-P 4675 4325
-F 0 "R25" V 4750 4275 50  0000 L CNN
-F 1 "10k" V 4675 4250 50  0000 L CNN
-F 2 "Resistors_SMD:R_0603_HandSoldering" V 4605 4325 50  0001 C CNN
-F 3 "~" H 4675 4325 50  0001 C CNN
-F 4 "1-0000010" H 4675 4325 50  0001 C CNN "Internal Part Number"
-F 5 "1" H 4675 4325 50  0001 C CNN "Populated"
-	1    4675 4325
+P 4100 4325
+F 0 "R25" V 4175 4275 50  0000 L CNN
+F 1 "10k" V 4100 4250 50  0000 L CNN
+F 2 "Resistors_SMD:R_0603_HandSoldering" V 4030 4325 50  0001 C CNN
+F 3 "~" H 4100 4325 50  0001 C CNN
+F 4 "1-0000010" H 4100 4325 50  0001 C CNN "Internal Part Number"
+F 5 "1" H 4100 4325 50  0001 C CNN "Populated"
+	1    4100 4325
 	1    0    0    -1
 $EndComp
@@
 L Device:R R26
 U 1 1 5DF776EE
-P 4825 4325
-F 0 "R26" V 4900 4275 50  0000 L CNN
-F 1 "10k" V 4825 4250 50  0000 L CNN
-F 2 "Resistors_SMD:R_0603_HandSoldering" V 4755 4325 50  0001 C CNN
-F 3 "~" H 4825 4325 50  0001 C CNN
-F 4 "1-0000010" H 4825 4325 50  0001 C CNN "Internal Part Number"
-F 5 "1" H 4825 4325 50  0001 C CNN "Populated"
-	1    4825 4325
+P 4250 4325
+F 0 "R26" V 4325 4275 50  0000 L CNN
+F 1 "10k" V 4250 4250 50  0000 L CNN
+F 2 "Resistors_SMD:R_0603_HandSoldering" V 4180 4325 50  0001 C CNN
+F 3 "~" H 4250 4325 50  0001 C CNN
+F 4 "1-0000010" H 4250 4325 50  0001 C CNN "Internal Part Number"
+F 5 "1" H 4250 4325 50  0001 C CNN "Populated"
+	1    4250 4325
 	1    0    0    -1
 $EndComp
 Wire Wire Line
-	4450 4525 4525 4525
+	3875 4525 3950 4525
 Wire Wire Line
-	4525 4525 4525 4475
+	3950 4525 3950 4475
 Wire Wire Line
-	4450 4625 4675 4625
+	3875 4625 4100 4625
 Wire Wire Line
-	4675 4625 4675 4475
+	4100 4625 4100 4475
 Wire Wire Line
-	4450 4725 4825 4725
+	3875 4725 4250 4725
 Wire Wire Line
-	4825 4725 4825 4475
+	4250 4725 4250 4475
 $Comp
 L power:+3V3 #PWR0110
 U 1 1 5DF82C74
-P 4675 4125
-F 0 "#PWR0110" H 4675 3975 50  0001 C CNN
-F 1 "+3V3" H 4690 4298 50  0000 C CNN
-F 2 "" H 4675 4125 50  0001 C CNN
-F 3 "" H 4675 4125 50  0001 C CNN
-	1    4675 4125
+P 4100 4125
+F 0 "#PWR0110" H 4100 3975 50  0001 C CNN
+F 1 "+3V3" H 4115 4298 50  0000 C CNN
+F 2 "" H 4100 4125 50  0001 C CNN
+F 3 "" H 4100 4125 50  0001 C CNN
+	1    4100 4125
 	1    0    0    -1
 $EndComp
@@
 L Switch:SW_DIP_x03 SW1
 U 1 1 5DF915C9
-P 4150 4725
-F 0 "SW1" H 4150 5192 50  0000 C CNN
-F 1 "Freq Select" H 4150 5101 50  0000 C CNN
-F 2 "lib_fp:KAE03TGGR" H 4150 4725 50  0001 C CNN
-F 3 "~" H 4150 4725 50  0001 C CNN
-F 4 "1-0000474" H 4150 4725 50  0001 C CNN "Internal Part Number"
-F 5 "1" H 4150 4725 50  0001 C CNN "Populated"
-	1    4150 4725
+P 3575 4725
+F 0 "SW1" H 3575 5192 50  0000 C CNN
+F 1 "Freq Select" H 3575 5101 50  0000 C CNN
+F 2 "lib_fp:KAE03TGGR" H 3575 4725 50  0001 C CNN
+F 3 "~" H 3575 4725 50  0001 C CNN
+F 4 "1-0000474" H 3575 4725 50  0001 C CNN "Internal Part Number"
+F 5 "1" H 3575 4725 50  0001 C CNN "Populated"
+	1    3575 4725
 	1    0    0    -1
 $EndComp
 Wire Wire Line
-	4525 4175 4525 4150
+	3950 4175 3950 4150
 Wire Wire Line
-	4525 4150 4675 4150
+	3950 4150 4100 4150
 Wire Wire Line
-	4825 4150 4825 4175
+	4250 4150 4250 4175
 Wire Wire Line
-	4675 4125 4675 4150
-Connection ~ 4675 4150
+	4100 4125 4100 4150
+Connection ~ 4100 4150
 Wire Wire Line
-	4675 4150 4825 4150
+	4100 4150 4250 4150
 Wire Wire Line
-	4675 4175 4675 4150
-Wire Wire Line
-	4525 4525 5325 4525
-Connection ~ 4525 4525
-Wire Wire Line
-	4675 4625 5325 4625
-Connection ~ 4675 4625
-Wire Wire Line
-	4825 4725 5325 4725
-Connection ~ 4825 4725
+	4100 4175 4100 4150
+Connection ~ 3950 4525
+Connection ~ 4100 4625
+Connection ~ 4250 4725
 $Comp
 L power:GND #PWR0111
 U 1 1 5DFAA612
-P 3800 4775
-F 0 "#PWR0111" H 3800 4525 50  0001 C CNN
-F 1 "GND" H 3805 4602 50  0000 C CNN
-F 2 "" H 3800 4775 50  0001 C CNN
-F 3 "" H 3800 4775 50  0001 C CNN
-	1    3800 4775
+P 3225 4775
+F 0 "#PWR0111" H 3225 4525 50  0001 C CNN
+F 1 "GND" H 3230 4602 50  0000 C CNN
+F 2 "" H 3225 4775 50  0001 C CNN
+F 3 "" H 3225 4775 50  0001 C CNN
+	1    3225 4775
 	-1   0    0    -1
 $EndComp
 Wire Wire Line
-	3800 4775 3800 4725
+	3225 4775 3225 4725
+Wire Wire Line
+	3225 4525 3275 4525
+Wire Wire Line
+	3275 4625 3225 4625
+Connection ~ 3225 4625
+Wire Wire Line
+	3225 4625 3225 4525
+Wire Wire Line
+	3275 4725 3225 4725
+Connection ~ 3225 4725
+Wire Wire Line
+	3225 4725 3225 4625
+Text Label 6625 3425 0    50   ~ 0
+Unused_Fiber_Ser_TX
+Text Label 5275 4150 2    50   ~ 0
+Unused_Radio_Ser_RX
+Wire Wire Line
+	5275 4150 5275 4125
+Wire Wire Line
+	5275 4125 5325 4125
 Wire Wire Line
-	3800 4525 3850 4525
+	3950 4525 5325 4525
 Wire Wire Line
-	3850 4625 3800 4625
-Connection ~ 3800 4625
+	4100 4625 5325 4625
 Wire Wire Line
-	3800 4625 3800 4525
+	4250 4725 5325 4725
+Text Label 12225 3775 0    50   ~ 0
+Unused_Fiber_Ser_TX
+Text Label 12225 3900 0    50   ~ 0
+Unused_Radio_Ser_RX
 Wire Wire Line
-	3850 4725 3800 4725
-Connection ~ 3800 4725
+	12225 3775 12150 3775
 Wire Wire Line
-	3800 4725 3800 4625
+	12225 3900 12150 3900
+NoConn ~ 12150 3900
+NoConn ~ 12150 3775
 $EndSCHEMATC
