File: Hardware/Control_PCB/KiCAD_Project/control_pcb/control_pcb.sch (KiCad schematic (older format))
At the start: 34 parts, among them J1 Conn_01x02, J2 ISP, J3 Spare, SW1 Freq Select, U1 STM32F103CBT6, Y1 8MHz

Commit message: Draft of next layout
Parts:
- removed C2, C3: 20pF, Capacitors_SMD:C_0603_HandSoldering, symbol Device:C
- removed FID3, FID4: Fiducial, Fiducials:Fiducial_0.75mm_Dia_1.5mm_Outer, symbol Mechanical:Fiducial
- removed R24, R25, R26: 10k, Resistors_SMD:R_0603_HandSoldering, symbol Device:R
- removed SW1: Freq Select, lib_fp:KAE03TGGR, symbol Switch:SW_DIP_x03
- removed Y1: 8MHz, Crystals:Crystal_SMD_HC49-SD_HandSoldering, symbol Device:Crystal
- added D1: Error, LED_SMD:LED_0805_2012Metric, symbol Device:LED
- added D2: Run, LED_SMD:LED_0805_2012Metric, symbol Device:LED
- added D3: Power, LED_SMD:LED_0805_2012Metric, symbol Device:LED
- added R11, R12, R18: 150, Resistor_SMD:R_0603_1608Metric, symbol Device:R
- added R13, R14: 1-0000006, resistors_0603:1-0000006, symbol resistors_0603:1-0000006
- added Y1: 8MHz, lib_fp:Resonator, symbol Device:Resonator_Small
- C1: renamed from C4; footprint Capacitors_SMD:C_0603_HandSoldering -> Capacitor_SMD:C_0603_1608Metric
- C2: renamed from C6; footprint Capacitors_SMD:C_0603_HandSoldering -> Capacitor_SMD:C_0603_1608Metric
- C3: renamed from C1; footprint Capacitors_SMD:C_0603_HandSoldering -> Capacitor_SMD:C_0603_1608Metric
- C4: renamed from C5; footprint Capacitors_SMD:C_0603_HandSoldering -> Capacitor_SMD:C_0603_1608Metric
- C5: renamed from C7; footprint Capacitors_SMD:C_0603_HandSoldering -> Capacitor_SMD:C_0603_1608Metric
- FID1, FID2: footprint Fiducials:Fiducial_0.75mm_Dia_1.5mm_Outer -> Fiducial:Fiducial_1mm_Mask2mm
- R1: renamed from R9; footprint Resistors_SMD:R_0603_HandSoldering -> Resistor_SMD:R_0603_1608Metric
- R10: renamed from R8; footprint Resistors_SMD:R_0603_HandSoldering -> Resistor_SMD:R_0603_1608Metric
- R2: renamed from R3; value 27k -> 18k; footprint Resistors_SMD:R_0603_HandSoldering -> Resistor_SMD:R_0603_1608Metric; Internal Part Number 1-0000078 -> 1-0000096
- R3: renamed from R4; footprint Resistors_SMD:R_0603_HandSoldering -> Resistor_SMD:R_0603_1608Metric
- R4: renamed from R5; footprint Resistors_SMD:R_0603_HandSoldering -> Resistor_SMD:R_0603_1608Metric
- R5: renamed from R7; footprint Resistors_SMD:R_0603_HandSoldering -> Resistor_SMD:R_0603_1608Metric
- R6: renamed from R10; footprint Resistors_SMD:R_0603_HandSoldering -> Resistor_SMD:R_0603_1608Metric
- R7: renamed from R1; footprint Resistors_SMD:R_0603_HandSoldering -> Resistor_SMD:R_0603_1608Metric
- R8: renamed from R2; footprint Resistors_SMD:R_0603_HandSoldering -> Resistor_SMD:R_0603_1608Metric
- R9: renamed from R6; footprint Resistors_SMD:R_0603_HandSoldering -> Resistor_SMD:R_0603_1608Metric
Connections:
- net labels added: RX_FROM_STM, TX_TO_STM
- net labels removed: Radio_Serial_Select, SD_CS, SD_DETECT, SPI1_MISO, SPI1_MOSI, SPI1_SCLK, TX_to_Radio, Unused_Radio_Ser_RX
- wire segments 107 -> 90
- no-connect marks 14 -> 20
Other:
- note added: "Setup to work with 2S batteries"
- note added: "The STM32 is the main controller, taking data from the rotating section via the\nfiber cable and GPS data, putting them in packets, and forwarding those. It can\nalso receive feedback from the SD controller if necessary, though currently\nnot needed."

Commit message: Add final production files
Parts:
- added PCB1: barepcb, lib_fp:barepcb, symbol lib_sch:barepcb
- renumbered R18 to R15
Changed lines of the file:
@@
 Sheet 1 6
 Title "Control Paddle Electronics - NSSL EFM"
-Date "2020-03-31"
-Rev "2.0"
+Date "2020-12-30"
+Rev "3.0"
 Comp "Leeman Geophysical LLC"
 Comment1 "(479) 373-3736"
@@
 	6725 1700 6725 1450
 $Comp
-L power:GND #PWR018
+L power:GND #PWR016
 U 1 1 5DF0B5C6
 P 5975 5025
-F 0 "#PWR018" H 5975 4775 50  0001 C CNN
+F 0 "#PWR016" H 5975 4775 50  0001 C CNN
 F 1 "GND" H 5980 4852 50  0000 C CNN
 F 2 "" H 5975 5025 50  0001 C CNN
@@
 $EndComp
 $Comp
-L power:GND #PWR021
+L power:GND #PWR019
 U 1 1 5DEED6CE
 P 6200 7425
-F 0 "#PWR021" H 6200 7175 50  0001 C CNN
+F 0 "#PWR019" H 6200 7175 50  0001 C CNN
 F 1 "GND" H 6205 7252 50  0000 C CNN
 F 2 "" H 6200 7425 50  0001 C CNN
@@
 Connection ~ 5000 2725
 $Comp
-L Device:R R18
+L Device:R R15
 U 1 1 5FFB081D
 P 10300 5950
-F 0 "R18" V 10225 5950 50  0000 C CNN
+F 0 "R15" V 10225 5950 50  0000 C CNN
 F 1 "150" V 10300 5950 50  0000 C CNN
 F 2 "Resistor_SMD:R_0603_1608Metric" V 10230 5950 50  0001 C CNN
@@
 $EndComp
 $Comp
-L power:GND #PWR020
+L power:GND #PWR018
 U 1 1 5FFB1939
 P 10750 5950
-F 0 "#PWR020" H 10750 5700 50  0001 C CNN
+F 0 "#PWR018" H 10750 5700 50  0001 C CNN
 F 1 "GND" H 10755 5777 50  0000 C CNN
 F 2 "" H 10750 5950 50  0001 C CNN
@@
 $EndComp
 $Comp
-L power:+3V3 #PWR019
+L power:+3V3 #PWR017
 U 1 1 5FFB5B5D
 P 10075 5950
-F 0 "#PWR019" H 10075 5800 50  0001 C CNN
+F 0 "#PWR017" H 10075 5800 50  0001 C CNN
 F 1 "+3V3" H 10090 6123 50  0000 C CNN
 F 2 "" H 10075 5950 50  0001 C CNN
@@
 NoConn ~ 5325 4625
 NoConn ~ 5325 4725
+$Comp
+L lib_sch:barepcb PCB1
+U 1 1 5FF42A98
+P 5750 7200
+F 0 "PCB1" H 5550 7050 50  0000 L CNN
+F 1 "barepcb" H 5600 7200 50  0000 L CNN
+F 2 "lib_fp:barepcb" H 5750 7200 50  0001 C CNN
+F 3 "" H 5750 7200 50  0001 C CNN
+F 4 "3-0000071" H 5750 7200 50  0001 C CNN "Internal Part Number"
+F 5 "1" H 5750 7200 50  0001 C CNN "Populated"
+	1    5750 7200
+	1    0    0    -1
+$EndComp
 $EndSCHEMATC

Commit message: Control Rev 3.1
Parts:
- D1: value Error -> GPS; footprint LED_SMD:LED_0805_2012Metric -> LED_THT:LED_D3.0mm_Horizontal_O1.27mm_Z2.0mm_Clear
- D2: value Run -> ACT; footprint LED_SMD:LED_0805_2012Metric -> LED_THT:LED_D3.0mm_Horizontal_O1.27mm_Z2.0mm_Clear
- D3: footprint LED_SMD:LED_0805_2012Metric -> LED_THT:LED_D3.0mm_Horizontal_O1.27mm_Z2.0mm_Clear
- PCB1: Internal Part Number 3-0000071 -> 3-0000112
Changed lines of the file:
@@
 Sheet 1 6
 Title "Control Paddle Electronics - NSSL EFM"
-Date "2020-12-30"
-Rev "3.0"
+Date "2021-11-22"
+Rev "3.1"
 Comp "Leeman Geophysical LLC"
 Comment1 "(479) 373-3736"
@@
 F 0 "D3" H 10593 5695 50  0000 C CNN
 F 1 "Power" H 10593 5786 50  0000 C CNN
-F 2 "LED_SMD:LED_0805_2012Metric" H 10600 5950 50  0001 C CNN
+F 2 "LED_THT:LED_D3.0mm_Horizontal_O1.27mm_Z2.0mm_Clear" H 10600 5950 50  0001 C CNN
 F 3 "~" H 10600 5950 50  0001 C CNN
 F 4 "1-0000598" H 10600 5950 50  0001 C CNN "Internal Part Number"
@@
 P 7675 3725
 F 0 "D1" H 7668 3470 50  0000 C CNN
-F 1 "Error" H 7668 3561 50  0000 C CNN
-F 2 "LED_SMD:LED_0805_2012Metric" H 7675 3725 50  0001 C CNN
+F 1 "GPS" H 7668 3561 50  0000 C CNN
+F 2 "LED_THT:LED_D3.0mm_Horizontal_O1.27mm_Z2.0mm_Clear" H 7675 3725 50  0001 C CNN
 F 3 "~" H 7675 3725 50  0001 C CNN
 F 4 "1-0000600" H 7675 3725 50  0001 C CNN "Internal Part Number"
@@
 P 7675 3900
 F 0 "D2" H 7675 4100 50  0000 C CNN
-F 1 "Run" H 7675 4000 50  0000 C CNN
-F 2 "LED_SMD:LED_0805_2012Metric" H 7675 3900 50  0001 C CNN
+F 1 "ACT" H 7675 4000 50  0000 C CNN
+F 2 "LED_THT:LED_D3.0mm_Horizontal_O1.27mm_Z2.0mm_Clear" H 7675 3900 50  0001 C CNN
 F 3 "~" H 7675 3900 50  0001 C CNN
 F 4 "1-0000598" H 7675 3900 50  0001 C CNN "Internal Part Number"
@@
 F 2 "lib_fp:barepcb" H 5750 7200 50  0001 C CNN
 F 3 "" H 5750 7200 50  0001 C CNN
-F 4 "3-0000071" H 5750 7200 50  0001 C CNN "Internal Part Number"
+F 4 "3-0000112" H 5750 7200 50  0001 C CNN "Internal Part Number"
 F 5 "1" H 5750 7200 50  0001 C CNN "Populated"
 	1    5750 7200
