File: Hardware/Control_PCB/KiCAD_Project/control_pcb/control_pcb.kicad_pcb (KiCad board)
At the start: 4 copper layers, 82.6 x 76.2 mm, 86 parts, among them J1 Conn_01x02, J2 ISP, J3 Spare, J5 Micro_SD_Card_Det, J6 Battery, J7 External Switch, Q1 BSS138, SW1 Freq Select, U1 STM32F103CBT6, U2 SN74LVC1G18, U3 TX2M-400-5-NSSL, U4 IF-D96F, U5 TC4S584F, U6 MAX-M8C, U7 LT1521-3.3, U8 MAX3232, Y1 8MHz

Commit message: Draft of next layout
Parts:
- removed AE1: Antenna_Shield, lib_fp:SMA
- removed FID3, FID4: Fiducial, Fiducials:Fiducial_0.75mm_Dia_1.5mm_Outer
- removed the J6 at (154.4, 116.8)
- removed the U7 at (146.7, 119.8)
- added D1: Error, LED_SMD:LED_0805_2012Metric, F.Cu at (134.1, 148.6)
- added D2: Run, LED_SMD:LED_0805_2012Metric, F.Cu at (134.1, 150.9)
- added D3: Power, LED_SMD:LED_0805_2012Metric, F.Cu at (140.2, 100.6)
- added D4: Activity, LED_SMD:LED_0805_2012Metric, F.Cu at (111.4, 143.8)
- added D5: Error, LED_SMD:LED_0805_2012Metric, F.Cu at (113.8, 143.8)
- added D6: Activity, LED_SMD:LED_0805_2012Metric, F.Cu at (104.0, 155.3)
- added D7: Error, LED_SMD:LED_0805_2012Metric, F.Cu at (107.3, 168.4)
- added D8: D_Schottky, Diode_SMD:D_SOD-123F, F.Cu at (131.9, 120.0)
- added J4: XBee ISP, Connector_PinHeader_2.54mm:PinHeader_2x04_P2.54mm_Vertical, F.Cu at (105.4, 148.8)
- added J5: XBee_uC_ISP, Connector_PinHeader_2.54mm:PinHeader_2x03_P2.54mm_Vertical, F.Cu at (122.6, 140.8)
- added J8: External Switch, Connector_PinHeader_2.54mm:PinHeader_1x02_P2.54mm_Vertical, F.Cu at (154.4, 124.5)
- added J9: Battery, Connector_PinHeader_2.54mm:PinHeader_1x02_P2.54mm_Vertical, F.Cu at (154.4, 116.8)
- added R31: 100k, Resistor_SMD:R_0603_1608Metric, F.Cu at (126.0, 154.2)
- added R32: NP, Resistor_SMD:R_0603_1608Metric, F.Cu at (127.6, 154.2)
- added R33: 100k, Resistor_SMD:R_0603_1608Metric, F.Cu at (130.7, 154.2)
- added R34: 100k, Resistor_SMD:R_0603_1608Metric, F.Cu at (132.3, 154.2)
- added R35: 100k, Resistor_SMD:R_0603_1608Metric, F.Cu at (134.0, 154.2)
- added R36: 150, Resistor_SMD:R_0603_1608Metric, F.Cu at (107.3, 166.4)
- added R37: 10k, Resistor_SMD:R_0603_1608Metric, F.Cu at (122.9, 105.7)
- added R38: 10k, Resistor_SMD:R_0603_1608Metric, F.Cu at (136.8, 110.0)
- added R39: 10k, Resistor_SMD:R_0603_1608Metric, F.Cu at (134.2, 104.0)
- added R40: 0R0, Resistor_SMD:R_0603_1608Metric, F.Cu at (132.5, 114.0)
- added R41: NP, Resistor_SMD:R_0603_1608Metric, F.Cu at (132.5, 112.4)
- added R42: 10, Resistor_SMD:R_0603_1608Metric, F.Cu at (94.5, 104.9)
- added R43: NP, Resistor_SMD:R_0603_1608Metric, F.Cu at (112.0, 114.2)
- added R44: 1-0000174, resistors_0603:1-0000174, F.Cu at (126.4, 116.1)
- added R45: 1-0000174, resistors_0603:1-0000174, F.Cu at (147.6, 104.4)
- added U4: ATmega328P-AU, Package_QFP:TQFP-32_7x7mm_P0.8mm, F.Cu at (111.4, 159.9)
- added U9: SPX3819M5-L-3-3, Package_TO_SOT_SMD:SOT-23-5, F.Cu at (144.3, 104.4)
- added Y2: 16MHz, lib_fp:Resonator, F.Cu at (108.8, 136.4)
- added Y3: 16MHz, lib_fp:Resonator, F.Cu at (104.0, 163.8)
- BT1: moved to B.Cu
- C1, C17: value 1u -> 0.1u; footprint Capacitors_SMD:C_0603_HandSoldering -> Capacitor_SMD:C_0603_1608Metric; moved to F.Cu
- C10: value 1u -> 10u; footprint Capacitors_SMD:C_0603_HandSoldering -> Capacitor_SMD:C_0603_1608Metric
- C11: value 0.1u -> 1u; footprint Capacitors_SMD:C_0603_HandSoldering -> Capacitor_SMD:C_0603_1608Metric; moved to F.Cu
- C12, C6, C7: value 0.1u -> 1-0000007; footprint Capacitors_SMD:C_0603_HandSoldering -> capacitors_0603:1-0000007; moved to F.Cu
- C13, C8: value 0.1u -> 1-0000007; footprint Capacitors_SMD:C_0603_HandSoldering -> capacitors_0603:1-0000007
- C14: value 47pF -> 1-0000007; footprint Capacitors_SMD:C_0603_HandSoldering -> capacitors_0603:1-0000007
- C15: value 10nF -> 1-0000007; footprint Capacitors_SMD:C_0603_HandSoldering -> capacitors_0603:1-0000007
- C16: value 10u -> 0.1u; footprint Capacitors_SMD:C_0603_HandSoldering -> Capacitor_SMD:C_0603_1608Metric; moved to F.Cu
- C18, C4, C5: footprint Capacitors_SMD:C_0603_HandSoldering -> Capacitor_SMD:C_0603_1608Metric; moved to F.Cu
- C19: value 10u -> 47pF; footprint Capacitors_SMD:C_0603_HandSoldering -> Capacitor_SMD:C_0603_1608Metric; moved to F.Cu
- C2: value 20pF -> 0.1u; footprint Capacitors_SMD:C_0603_HandSoldering -> Capacitor_SMD:C_0603_1608Metric; moved to F.Cu
- C20: value 1u -> 10nF; footprint Capacitors_SMD:C_0603_HandSoldering -> Capacitor_SMD:C_0603_1608Metric; moved to F.Cu
- C21, C24, C25: value 0.1u -> 1-0000075; footprint Capacitors_SMD:C_0603_HandSoldering -> capacitors_0805:1-0000075; moved to F.Cu
- C22: value 0.1u -> 1-0000075; footprint Capacitors_SMD:C_0603_HandSoldering -> capacitors_0805:1-0000075
- C23, C26: value 0.1u -> 1-0000018; footprint Capacitors_SMD:C_0603_HandSoldering -> capacitors_0603:1-0000018; moved to F.Cu
- C3: value 20pF -> 1u; footprint Capacitors_SMD:C_0603_HandSoldering -> Capacitor_SMD:C_0603_1608Metric; moved to F.Cu
- C9: value 10u -> 1-0000007; footprint Capacitors_SMD:C_0603_HandSoldering -> capacitors_0603:1-0000007
- FID1, FID2: footprint Fiducials:Fiducial_0.75mm_Dia_1.5mm_Outer -> Fiducial:Fiducial_1mm_Mask2mm
- J7: value External Switch -> SD_uC_ISP; footprint Pin_Headers:Pin_Header_Straight_1x02_Pitch2.54mm -> Connector_PinHeader_2.54mm:PinHeader_2x03_P2.54mm_Vertical
- R1, R15, R16, R17: value 100k -> 10k; footprint Resistors_SMD:R_0603_HandSoldering -> Resistor_SMD:R_0603_1608Metric; moved to F.Cu
- R10: value 1M -> 0R0; footprint Resistors_SMD:R_0603_HandSoldering -> Resistor_SMD:R_0603_1608Metric; moved to F.Cu
- R11, R12: value 100k -> 150; footprint Resistors_SMD:R_0603_HandSoldering -> Resistor_SMD:R_0603_1608Metric; moved to F.Cu
- R13: value 100k -> 1-0000006; footprint Resistors_SMD:R_0603_HandSoldering -> resistors_0603:1-0000006; moved to F.Cu
- R14: value NP -> 1-0000006; footprint Resistors_SMD:R_0603_HandSoldering -> resistors_0603:1-0000006; moved to F.Cu
- R18: value NP -> 150; footprint Resistors_SMD:R_0603_HandSoldering -> Resistor_SMD:R_0603_1608Metric
- R19: value 0R0 -> 1-0000010; footprint Resistors_SMD:R_0603_HandSoldering -> resistors_0603:1-0000010
- R2: value 100k -> 18k; footprint Resistors_SMD:R_0603_HandSoldering -> Resistor_SMD:R_0603_1608Metric; moved to F.Cu
- R20: value NP -> 1-0000006; footprint Resistors_SMD:R_0603_HandSoldering -> resistors_0603:1-0000006
- R21: value 10 -> 1-0000006; footprint Resistors_SMD:R_1218_HandSoldering -> resistors_0603:1-0000006
- R22, R26, R27: value 10k -> 1-0000006; footprint Resistors_SMD:R_0603_HandSoldering -> resistors_0603:1-0000006; moved to F.Cu
- R23, R24: value 10k -> 150; footprint Resistors_SMD:R_0603_HandSoldering -> Resistor_SMD:R_0603_1608Metric; moved to F.Cu
- R25: value 10k -> 1-0000010; footprint Resistors_SMD:R_0603_HandSoldering -> resistors_0603:1-0000010; moved to F.Cu
- R28: value 10k -> 150; footprint Resistors_SMD:R_0603_HandSoldering -> Resistor_SMD:R_0603_1608Metric
- R29: value 10k -> 100k; footprint Resistor_SMD:R_0603_1608Metric_Pad1.05x0.95mm_HandSolder -> Resistor_SMD:R_0603_1608Metric; moved to F.Cu
- R3: value 27k -> 10k; footprint Resistors_SMD:R_0603_HandSoldering -> Resistor_SMD:R_0603_1608Metric; moved to F.Cu
- R30: value NP -> 100k; footprint Resistor_SMD:R_0603_1608Metric_Pad1.05x0.95mm_HandSolder -> Resistor_SMD:R_0603_1608Metric
- R4: value 10k -> NP; footprint Resistors_SMD:R_0603_HandSoldering -> Resistor_SMD:R_0603_1608Metric; moved to F.Cu
- R5: footprint Resistors_SMD:R_0603_HandSoldering -> Resistor_SMD:R_0603_1608Metric; moved to F.Cu
- R6: value 0R0 -> 1M; footprint Resistors_SMD:R_0603_HandSoldering -> Resistor_SMD:R_0603_1608Metric; moved to F.Cu
- R7: value NP -> 100k; footprint Resistors_SMD:R_0603_HandSoldering -> Resistor_SMD:R_0603_1608Metric; moved to F.Cu
- R8: value 0R0 -> 100k; footprint Resistors_SMD:R_0603_HandSoldering -> Resistor_SMD:R_0603_1608Metric; moved to F.Cu
- R9: value 10k -> 0R0; footprint Resistors_SMD:R_0603_HandSoldering -> Resistor_SMD:R_0603_1608Metric; moved to F.Cu
- SW1: value Freq Select -> ID Select
- U2: value SN74LVC1G18 -> ATmega328P-AU; footprint lib_fp:SN74LVC1G18DCKR -> Package_QFP:TQFP-32_7x7mm_P0.8mm
- U3: value TX2M-400-5-NSSL -> XTend; footprint lib_fp:TX2M -> lib_fp:XTend; moved to F.Cu
- U8: value MAX3232 -> SPX3819M5-L-3-3; footprint Housings_SSOP:TSSOP-16_4.4x5mm_Pitch0.65mm -> Package_TO_SOT_SMD:SOT-23-5
- Y1: footprint Crystals:Crystal_SMD_HC49-SD_HandSoldering -> lib_fp:Resonator
- moved FID1 78.0 mm to (154.2, 106.7)
- moved R28 61.4 mm to (104.0, 157.5), turned to 0 degrees
- moved R30 61.3 mm to (124.3, 154.2), turned to 90 degrees
- moved C12 59.4 mm to (104.0, 159.1), turned to 180 degrees
- moved AE2 58.7 mm to (87.5, 108.5), turned to 180 degrees
- moved J7 56.9 mm to (117.6, 167.8), turned to 270 degrees
- moved R27 50.9 mm to (109.0, 152.7), turned to 270 degrees
- moved L1 50.8 mm to (94.4, 108.5), turned to 0 degrees
- moved C13 49.5 mm to (118.7, 162.2), turned to 0 degrees
- moved R29 48.2 mm to (135.6, 154.2)
- moved C19 46.9 mm to (94.4, 110.1), turned to 0 degrees
- moved C20 45.9 mm to (94.4, 106.8), turned to 0 degrees
- moved R26 37.0 mm to (110.7, 152.7), turned to 270 degrees
- moved U7 36.8 mm to (103.1, 113.4), turned to 180 degrees
- moved C16 34.4 mm to (129.2, 154.3)
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- renumbered J5 to J6, U4 to U5, U5 to U6, U6 to U7
Connections:
- C1 pad 1: /Reset -> GND
- C1 pad 2: GND -> +3V3
- C10 pad 1: +BATT -> 3V3_XBEE
- C11 pad 1: GND -> 3V3_XBEE
- C11 pad 2: +3V3 -> GND
- C12 pad 1: +BATT -> +3V3
- C13 pad 1: +BATT -> +3V3
- C14 pad 1: Net-(AE2-Pad1) -> +3V3
- C14 pad 2: Net-(C14-Pad2) -> GND
- C15 pad 1: GND -> Net-(C15-Pad1)
- C15 pad 2: Net-(C15-Pad2) -> GND
- C16 pad 1: +BATT -> GND
- C16 pad 2: GND -> +3V3
- C19 pad 1: +3V3 -> Net-(AE2-Pad1)
- C19 pad 2: GND -> Net-(C19-Pad2)
- C2 pad 1: Net-(C2-Pad1) -> GND
- C2 pad 2: GND -> +3V3
- C20 pad 1: +3V3 -> GND
- C20 pad 2: GND -> Net-(C20-Pad2)
- C21 pad 1: +3V3 -> Net-(C21-Pad1)
- C22 pad 1: Net-(C22-Pad1) -> +3V3
- C22 pad 2: Net-(C22-Pad2) -> GND
- C23 pad 1: GND -> +3V3
- C23 pad 2: +3V3 -> GND
- C24 pad 1: Net-(C24-Pad1) -> Net-(C21-Pad1)
- C24 pad 2: Net-(C24-Pad2) -> GND
- C25 pad 1: GND -> 3V3_XBEE
- C25 pad 2: Net-(C25-Pad2) -> GND
- C26 pad 1: GND -> 3V3_XBEE
- C26 pad 2: Net-(C26-Pad2) -> GND
- C3 pad 1: Net-(C3-Pad1) -> /Reset
- C6 pad 1: GND -> +3V3
- C6 pad 2: +3V3 -> GND
- C7 pad 1: GND -> +3V3
- C7 pad 2: +3V3 -> GND
- C9 pad 1: +BATT -> Net-(C9-Pad1)
- J6 pad 1: Net-(J5-Pad1) -> Net-(J6-Pad1)
- J6 pad 2: SD_CS -> /SD/SD_uC_CS
- J6 pad 3: SPI1_MOSI -> /SD/SD_uC_MOSI
- J6 pad 5: SPI1_SCLK -> /SD/SD_uC_SCK
- J6 pad 7: SPI1_MISO -> /SD/SD_uC_MISO
- J6 pad 8: Net-(J5-Pad8) -> Net-(J6-Pad8)
- J6 pad 9: SD_DETECT -> /SD/SD_uC_CD
- J7 pad 1: Net-(F1-Pad2) -> /SD/SD_uC_MISO
- J7 pad 2: Net-(J6-Pad1) -> +3V3
- L1 pad 2: Net-(C15-Pad2) -> Net-(C20-Pad2)
- R1 pad 1: Net-(R1-Pad1) -> +3V3
- R1 pad 2: /Boot0 -> /Reset
- R10 pad 1: Net-(C2-Pad1) -> GND
- R10 pad 2: Net-(C3-Pad1) -> Net-(R10-Pad2)
- R11 pad 1: +3V3 -> Net-(D1-Pad2)
- R11 pad 2: SD_DETECT -> Net-(R11-Pad2)
- R12 pad 1: +3V3 -> Net-(D2-Pad2)
- R12 pad 2: Net-(J5-Pad8) -> Net-(R12-Pad2)
- R13 pad 1: +3V3 -> Net-(R13-Pad1)
- R13 pad 2: SPI1_MISO -> RX_FROM_STM
- R14 pad 1: +3V3 -> Net-(R14-Pad1)
- R14 pad 2: SPI1_SCLK -> TX_TO_STM
- R15 pad 2: SPI1_MOSI -> Net-(R15-Pad2)
- R16 pad 2: SD_CS -> Net-(R16-Pad2)
- R17 pad 2: Net-(J5-Pad1) -> Net-(R17-Pad2)
- R18 pad 1: Net-(Q1-Pad3) -> Net-(D3-Pad2)
- R18 pad 2: Net-(R18-Pad2) -> +3V3
- R19 pad 1: Net-(Q1-Pad3) -> +3V3
- R19 pad 2: Net-(R19-Pad2) -> /radio/XBEE_uC_RESET
- R2 pad 1: Net-(R2-Pad1) -> +BATT
- R2 pad 2: /Boot1 -> /VBat_Sense
- R20 pad 1: GPS_PPS -> RX_FROM_STM
- R20 pad 2: +3V3 -> Net-(R20-Pad2)
- R21 pad 1: +3V3 -> RX_FROM_RADIO
- R21 pad 2: Net-(C15-Pad2) -> Net-(R21-Pad2)
- R22 pad 1: GND -> TX_TO_RADIO
- R23 pad 1: GND -> Net-(D4-Pad2)
- R24 pad 1: +3V3 -> Net-(D5-Pad2)
- R25 pad 2: Net-(R25-Pad2) -> /SD/SD_uC_RESET
- R26 pad 1: +3V3 -> RX_FROM_STM
- R27 pad 1: +BATT -> TX_TO_STM
- R27 pad 2: Net-(Q1-Pad3) -> Net-(R27-Pad2)
- R28 pad 1: +3V3 -> Net-(D6-Pad2)
- R28 pad 2: Fiber_Serial_In -> Net-(R28-Pad2)
- R29 pad 1: +BATT -> +3V3
- R29 pad 2: Net-(R19-Pad2) -> /SD/SD_uC_CD
- R3 pad 1: +BATT -> /VBat_Sense
- R3 pad 2: /VBat_Sense -> GND
- R30 pad 1: GND -> +3V3
- R30 pad 2: Net-(R30-Pad2) -> Net-(J6-Pad8)
- R4 pad 1: /VBat_Sense -> Net-(R4-Pad1)
- R4 pad 2: GND -> +3V3
- R5 pad 1: Net-(R1-Pad1) -> Net-(R10-Pad2)
- R6 pad 1: GND -> Net-(R6-Pad1)
- R6 pad 2: Net-(R1-Pad1) -> Net-(R6-Pad2)
- R7 pad 1: Net-(R2-Pad1) -> Net-(R4-Pad1)
- R7 pad 2: +3V3 -> /Boot0
- R8 pad 1: GND -> Net-(R10-Pad2)
- R8 pad 2: Net-(R2-Pad1) -> /Boot1
- R9 pad 1: +3V3 -> GND
- R9 pad 2: /Reset -> Net-(R4-Pad1)
- SW1 pad 4: Net-(R26-Pad2) -> Net-(R15-Pad2)
- SW1 pad 5: Net-(R25-Pad2) -> Net-(R16-Pad2)
- SW1 pad 6: Net-(R24-Pad2) -> Net-(R17-Pad2)
- U1 pad 15: SPI1_SCLK -> Net-(R11-Pad2)
- U1 pad 16: SPI1_MISO -> Net-(R12-Pad2)
- U1 pad 17: SPI1_MOSI -> (no net)
- U1 pad 20: Radio_Serial_Select -> (no net)
- U1 pad 21: (no net) -> Net-(R13-Pad1)
- U1 pad 22: (no net) -> Net-(R14-Pad1)
- U1 pad 26: Net-(R24-Pad2) -> (no net)
- U1 pad 27: Net-(R25-Pad2) -> (no net)
- U1 pad 28: Net-(R26-Pad2) -> (no net)
- U1 pad 29: SD_DETECT -> (no net)
- U1 pad 32: SD_CS -> (no net)
- U1 pad 45: TX_to_Radio -> (no net)
- U1 pad 5: Net-(C2-Pad1) -> Net-(R6-Pad1)
- U1 pad 6: Net-(C3-Pad1) -> Net-(R6-Pad2)
- U2 pad 1: Radio_Serial_Select -> Net-(R22-Pad2)
- U2 pad 2: GND -> (no net)
- U2 pad 3: TX_to_Radio -> GND
- U2 pad 4: Net-(U2-Pad4) -> +3V3
- U2 pad 5: +3V3 -> GND
- U2 pad 6: Net-(U2-Pad6) -> +3V3
- U5 pad 2: Net-(R19-Pad2) -> Net-(R37-Pad2)
- U6 pad 2: Net-(R19-Pad2) -> Net-(R37-Pad2)
- U6 pad 4: Net-(R18-Pad2) -> Net-(R40-Pad2)
- U7 pad 11: Net-(C14-Pad2) -> Net-(C19-Pad2)
- U8 pad 1: Net-(C22-Pad1) -> Net-(C21-Pad1)
- U8 pad 2: Net-(C25-Pad2) -> GND
- U8 pad 3: Net-(C22-Pad2) -> Net-(R44-Pad2)
- U8 pad 4: Net-(C24-Pad1) -> (no net)
- U8 pad 5: Net-(C24-Pad2) -> +3V3
- Y1 pad 1: Net-(C2-Pad1) -> Net-(R6-Pad1)
- Y1 pad 2: Net-(C3-Pad1) -> GND
Routing:
- net 3V3_XBEE: track 0.00 -> 165.0 mm, vias 0 -> 6
- net Net-(R16-Pad2): track 0.00 -> 68.7 mm, vias 0 -> 4
- net Net-(R15-Pad2): track 0.00 -> 67.9 mm, vias 0 -> 2
- net TX_to_Radio: track 67.0 -> 0.00 mm, vias 2 -> 0
- net Net-(R17-Pad2): track 0.00 -> 65.4 mm, vias 0 -> 4
- net Radio_Serial_Select: track 63.9 -> 0.00 mm, vias 2 -> 0
- net RX_FROM_STM: track 0.00 -> 57.9 mm, vias 0 -> 3
- net +BATT: track 118.3 -> 70.7 mm, vias 3 -> 2
- net SD_CS: track 46.6 -> 0.00 mm, vias 5 -> 0
- net /SD/SD_uC_MOSI: track 0.00 -> 45.7 mm, vias 0 -> 2
- net /SD/SD_uC_CS: track 0.00 -> 45.0 mm, vias 0 -> 4
- net GND: track 68.4 -> 112.4 mm, vias 35 -> 63
- net /radio/Data_RS232: track 42.2 -> 0.00 mm
- net /radio/Programming_RS232: track 42.0 -> 0.00 mm
- net SD_DETECT: track 39.8 -> 0.00 mm, vias 5 -> 0
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- removed copper zone on B.Cu, net GND
Other:
- board text added: "Act"
- board text added: "Err"
- board text added: "ID"
- board text added: "PWR"
- board text added: "Run"
- board text removed: "FREQ"
- board text removed: "Radio"

Commit message: Add final production files
Parts:
- added PCB1: barepcb, lib_fp:barepcb, F.Cu at (180.8, 160.5)
- renumbered AE2 to AE1, R18 to R15, R19 to R16, R15 to R17, R16 to R18, R17 to R19, U3 to U2, U2 to U3
Other:
- rule pad_to_mask_clearance: 0.0508 -> 0
- board text added: "Data Control Module Rev 3.0 P/N 3-0000071"
- board text removed: "Data Control Module Rev 2.0 April 2020 P/N 3-0000032"

Commit message: Control PCB hardware updates
Other:
- board text added: "*"
- board text added: "3V3"
- board text added: "BATT"
- board text added: "G"
- board text added: "GND"
- board text added: "PB3"
- board text added: "PB4"
- board text added: "PB5"
- board text added: "PB6"
- board text added: "SWCLK"
- board text added: "SWDIO"
- board text added: "Switch"
