File: Hardware/Control_PCB/KiCAD_Project/control_pcb/control_pcb.kicad_pcb (KiCad board)
At the start: 4 copper layers, 82.6 x 76.2 mm, 113 parts, among them J1 Conn_01x02, J2 ISP, J3 Spare, J4 XBee ISP, J5 XBee_uC_ISP, J6 Micro_SD_Card_Det, J7 SD_uC_ISP, J8 External Switch, J9 Battery, Q1 BSS138, SW1 ID Select, U1 STM32F103CBT6, U2 XTend, U3 ATmega328P-AU, U4 ATmega328P-AU, U5 IF-D96F, U6 TC4S584F, U7 MAX-M8C, U8 SPX3819M5-L-3-3, U9 SPX3819M5-L-3-3, Y1 8MHz, Y2 16MHz, Y3 16MHz

Commit message: Control Rev 3.1
Parts:
- removed R45: 1-0000174, resistors_0603:1-0000174
- D1: value Error -> GPS; footprint LED_SMD:LED_0805_2012Metric -> LED_THT:LED_D3.0mm_Horizontal_O1.27mm_Z2.0mm_Clear
- D2: value Run -> ACT; footprint LED_SMD:LED_0805_2012Metric -> LED_THT:LED_D3.0mm_Horizontal_O1.27mm_Z2.0mm_Clear
- D3, D4, D5, D6, D7: footprint LED_SMD:LED_0805_2012Metric -> LED_THT:LED_D3.0mm_Horizontal_O1.27mm_Z2.0mm_Clear
- U9: value SPX3819M5-L-3-3 -> 1-0000946; footprint Package_TO_SOT_SMD:SOT-23-5 -> dc_dc_converters:1-0000946
- Y2, Y3: value 16MHz -> 8MHz
- moved C25 61.5 mm to (80.0, 112.4), turned to 180 degrees
- moved U9 61.3 mm to (84.8, 119.6)
- moved C26 59.3 mm to (80.0, 110.5), turned to 180 degrees
- moved D6 51.3 mm to (153.9, 167.0), turned to 90 degrees
- moved C24 49.3 mm to (97.0, 121.5), turned to 270 degrees
- moved D7 47.1 mm to (153.9, 161.9), turned to 90 degrees
- moved D4 44.5 mm to (153.9, 156.8)
- moved D5 40.9 mm to (153.9, 151.8)
- moved D1 21.0 mm to (153.9, 141.6), turned to 90 degrees
- moved D2 20.3 mm to (153.9, 146.7), turned to 90 degrees
- moved J3 6.35 mm to (154.4, 128.3)
- moved H3 2.92 mm to (149.5, 168.9)
- moved D3 2.84 mm to (141.5, 98.0), turned to 180 degrees
Connections:
- U9 pad 1: Net-(C21-Pad1) -> GND
- U9 pad 2: GND -> Net-(C21-Pad1)
- U9 pad 3: Net-(R45-Pad2) -> (no net)
- U9 pad 5: 3V3_XBEE -> (no net)
Routing:
- net 3V3_XBEE: track 165.0 -> 60.2 mm, vias 6 -> 2
- net Net-(D6-Pad2): track 2.21 -> 70.7 mm, vias 0 -> 1
- net Net-(D7-Pad2): track 2.08 -> 58.3 mm
- net Net-(D4-Pad2): track 1.92 -> 50.8 mm, vias 0 -> 2
- net Net-(D5-Pad2): track 1.92 -> 46.0 mm, vias 0 -> 2
- net Net-(D1-Pad2): track 2.15 -> 27.6 mm, vias 0 -> 2
- net Net-(D2-Pad2): track 2.15 -> 26.4 mm, vias 0 -> 2
- net Net-(C21-Pad1): track 31.9 -> 47.8 mm, vias 4 -> 0
- net GND: track 112.4 -> 103.1 mm, vias 63 -> 57
- net Net-(J3-Pad1): track 16.3 -> 22.4 mm, vias 1 -> 2
- net Net-(J3-Pad4): track 19.2 -> 13.6 mm, vias 2 -> 1
- net Net-(D3-Pad2): track 1.79 -> 5.05 mm
- net Net-(J3-Pad2): track 17.0 -> 19.5 mm
- net Net-(R45-Pad2): track 2.27 -> 0.00 mm
- net Net-(J3-Pad3): track 18.4 -> 16.6 mm
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Other:
- board text added: "Data Control Module Rev 3.1 P/N 3-0000112"
- board text added: "M ACT"
- board text added: "SD ACT"
- board text added: "SD Err"
- board text added: "XB ACT"
- board text added: "XB ERR"
- board text removed: "Act"
- board text removed: "Data Control Module Rev 3.0 P/N 3-0000071"
- board text removed: "Err"
- board text removed: "Run"
