File: Hardware/Control_PCB/KiCAD_Project/control_pcb/GPS.sch (KiCad schematic (older format))
At the start: 8 parts, among them U6 MAX-M8C

Commit message: Draft of next layout
Parts:
- C19: renamed from C14; footprint Capacitors_SMD:C_0603_HandSoldering -> Capacitor_SMD:C_0603_1608Metric
- C20: renamed from C15; footprint Capacitors_SMD:C_0603_HandSoldering -> Capacitor_SMD:C_0603_1608Metric
- R42: renamed from R21; footprint Resistors_SMD:R_1218_HandSoldering -> Resistor_SMD:R_0603_1608Metric
- R43: renamed from R20; footprint Resistors_SMD:R_0603_HandSoldering -> Resistor_SMD:R_0603_1608Metric
- renumbered U6 to U7
Other:
- note added: "Active antenna GPS receiver sends GPS packets via serial to the STM32."
Changed lines of the file:
@@
 $EndDescr
 $Comp
-L RF_GPS:MAX-M8C U6
+L RF_GPS:MAX-M8C U7
 U 1 1 5DF754E8
 P 5425 3525
-F 0 "U6" H 5875 2800 50  0000 C CNN
+F 0 "U7" H 5875 2800 50  0000 C CNN
 F 1 "MAX-M8C" H 5750 2875 50  0000 C CNN
 F 2 "lib_fp:XCVR_MAX-M8C-0-10" H 5825 2875 50  0001 C CNN
@@
 Antenna\n1-0000457
 $Comp
-L Device:C C14
+L Device:C C19
 U 1 1 5DF75D28
 P 6750 3525
-F 0 "C14" V 6498 3525 50  0000 C CNN
+F 0 "C19" V 6498 3525 50  0000 C CNN
 F 1 "47pF" V 6589 3525 50  0000 C CNN
-F 2 "Capacitors_SMD:C_0603_HandSoldering" H 6788 3375 50  0001 C CNN
+F 2 "Capacitor_SMD:C_0603_1608Metric" H 6788 3375 50  0001 C CNN
 F 3 "~" H 6750 3525 50  0001 C CNN
 F 4 "1-0000458" H 6750 3525 50  0001 C CNN "Internal Part Number"
@@
 $EndComp
 $Comp
-L Device:C C15
+L Device:C C20
 U 1 1 5DF760F7
 P 7000 4325
-F 0 "C15" H 6885 4279 50  0000 R CNN
+F 0 "C20" H 6885 4279 50  0000 R CNN
 F 1 "10nF" H 6885 4370 50  0000 R CNN
-F 2 "Capacitors_SMD:C_0603_HandSoldering" H 7038 4175 50  0001 C CNN
+F 2 "Capacitor_SMD:C_0603_1608Metric" H 7038 4175 50  0001 C CNN
 F 3 "~" H 7000 4325 50  0001 C CNN
 F 4 "1-0000014" H 7000 4325 50  0001 C CNN "Internal Part Number"
@@
 $EndComp
 $Comp
-L Device:R R21
+L Device:R R42
 U 1 1 5DF763A0
 P 7275 4125
-F 0 "R21" V 7200 4125 50  0000 C CNN
+F 0 "R42" V 7200 4125 50  0000 C CNN
 F 1 "10" V 7275 4125 50  0000 C CNN
-F 2 "Resistors_SMD:R_1218_HandSoldering" V 7205 4125 50  0001 C CNN
+F 2 "Resistor_SMD:R_0603_1608Metric" V 7205 4125 50  0001 C CNN
 F 3 "~" H 7275 4125 50  0001 C CNN
 F 4 "1-0000460" H 7275 4125 50  0001 C CNN "Internal Part Number"
@@
 $EndComp
 $Comp
-L power:+3V3 #PWR038
+L power:+3V3 #PWR060
 U 1 1 5DF79241
 P 7525 4100
-F 0 "#PWR038" H 7525 3950 50  0001 C CNN
+F 0 "#PWR060" H 7525 3950 50  0001 C CNN
 F 1 "+3V3" H 7540 4273 50  0000 C CNN
 F 2 "" H 7525 4100 50  0001 C CNN
@@
 Connection ~ 7000 3525
 $Comp
-L power:GND #PWR039
+L power:GND #PWR059
 U 1 1 5DF7AF66
 P 7850 3525
-F 0 "#PWR039" H 7850 3275 50  0001 C CNN
+F 0 "#PWR059" H 7850 3275 50  0001 C CNN
 F 1 "GND" H 7855 3352 50  0000 C CNN
 F 2 "" H 7850 3525 50  0001 C CNN
@@
 $EndComp
 $Comp
-L power:GND #PWR037
+L power:GND #PWR062
 U 1 1 5DF7B3E0
 P 7000 4475
-F 0 "#PWR037" H 7000 4225 50  0001 C CNN
+F 0 "#PWR062" H 7000 4225 50  0001 C CNN
 F 1 "GND" H 7005 4302 50  0000 C CNN
 F 2 "" H 7000 4475 50  0001 C CNN
@@
 $EndComp
 $Comp
-L power:GND #PWR035
+L power:GND #PWR061
 U 1 1 5DF7B7C2
 P 5425 4225
-F 0 "#PWR035" H 5425 3975 50  0001 C CNN
+F 0 "#PWR061" H 5425 3975 50  0001 C CNN
 F 1 "GND" H 5430 4052 50  0000 C CNN
 F 2 "" H 5425 4225 50  0001 C CNN
@@
 $EndComp
 $Comp
-L power:+3V3 #PWR034
+L power:+3V3 #PWR057
 U 1 1 5DF7BDF6
 P 5225 2525
-F 0 "#PWR034" H 5225 2375 50  0001 C CNN
+F 0 "#PWR057" H 5225 2375 50  0001 C CNN
 F 1 "+3V3" H 5240 2698 50  0000 C CNN
 F 2 "" H 5225 2525 50  0001 C CNN
@@
 	5425 2525 5425 2825
 $Comp
-L power:GND #PWR036
+L power:GND #PWR058
 U 1 1 5DF80C9B
 P 5725 2525
-F 0 "#PWR036" H 5725 2275 50  0001 C CNN
+F 0 "#PWR058" H 5725 2275 50  0001 C CNN
 F 1 "GND" H 5730 2352 50  0000 C CNN
 F 2 "" H 5725 2525 50  0001 C CNN
@@
 GPS_PPS
 $Comp
-L Device:R R20
+L Device:R R43
 U 1 1 5DF84FAE
 P 5225 5100
-F 0 "R20" V 5150 5100 50  0000 C CNN
+F 0 "R43" V 5150 5100 50  0000 C CNN
 F 1 "NP" V 5225 5100 50  0000 C CNN
-F 2 "Resistors_SMD:R_0603_HandSoldering" V 5155 5100 50  0001 C CNN
+F 2 "Resistor_SMD:R_0603_1608Metric" V 5155 5100 50  0001 C CNN
 F 3 "~" H 5225 5100 50  0001 C CNN
 F 4 "1-0000010" H 5225 5100 50  0001 C CNN "Internal Part Number"
@@
 $EndComp
 $Comp
-L power:+3V3 #PWR033
+L power:+3V3 #PWR063
 U 1 1 5DF854B1
 P 5075 5100
-F 0 "#PWR033" H 5075 4950 50  0001 C CNN
+F 0 "#PWR063" H 5075 4950 50  0001 C CNN
 F 1 "+3V3" H 5090 5273 50  0000 C CNN
 F 2 "" H 5075 5100 50  0001 C CNN
@@
 $EndBitmap
 $Comp
-L power:PWR_FLAG #FLG0102
+L power:PWR_FLAG #FLG03
 U 1 1 5DEB3E01
 P 5425 2525
-F 0 "#FLG0102" H 5425 2600 50  0001 C CNN
+F 0 "#FLG03" H 5425 2600 50  0001 C CNN
 F 1 "PWR_FLAG" V 5425 2825 50  0000 C CNN
 F 2 "" H 5425 2525 50  0001 C CNN
@@
 $EndComp
 Connection ~ 5425 2525
+Text Notes 8200 650  0    50   ~ 0
+Active antenna GPS receiver sends GPS packets via serial to the STM32.
 $EndSCHEMATC

Commit message: Add final production files
Parts:
- renumbered AE2 to AE1
Changed lines of the file:
@@
 Sheet 5 6
 Title "Control Paddle Electronics - NSSL EFM"
-Date "2020-03-31"
-Rev "2.0"
+Date "2020-12-30"
+Rev "3.0"
 Comp "Leeman Geophysical LLC"
 Comment1 "(479) 373-3736"
@@
 $EndComp
 $Comp
-L power:+3V3 #PWR060
+L power:+3V3 #PWR058
 U 1 1 5DF79241
 P 7525 4100
-F 0 "#PWR060" H 7525 3950 50  0001 C CNN
+F 0 "#PWR058" H 7525 3950 50  0001 C CNN
 F 1 "+3V3" H 7540 4273 50  0000 C CNN
 F 2 "" H 7525 4100 50  0001 C CNN
@@
 	6600 3525 6025 3525
 $Comp
-L Device:Antenna_Shield AE2
+L Device:Antenna_Shield AE1
 U 1 1 5DF79EDC
 P 7750 3325
-F 0 "AE2" H 7894 3364 50  0000 L CNN
+F 0 "AE1" H 7894 3364 50  0000 L CNN
 F 1 "Antenna_Shield" H 7894 3273 50  0001 L CNN
 F 2 "lib_fp:SMA" H 7750 3425 50  0001 C CNN
@@
 Connection ~ 7000 3525
 $Comp
-L power:GND #PWR059
+L power:GND #PWR057
 U 1 1 5DF7AF66
 P 7850 3525
-F 0 "#PWR059" H 7850 3275 50  0001 C CNN
+F 0 "#PWR057" H 7850 3275 50  0001 C CNN
 F 1 "GND" H 7855 3352 50  0000 C CNN
 F 2 "" H 7850 3525 50  0001 C CNN
@@
 $EndComp
 $Comp
-L power:GND #PWR062
+L power:GND #PWR060
 U 1 1 5DF7B3E0
 P 7000 4475
-F 0 "#PWR062" H 7000 4225 50  0001 C CNN
+F 0 "#PWR060" H 7000 4225 50  0001 C CNN
 F 1 "GND" H 7005 4302 50  0000 C CNN
 F 2 "" H 7000 4475 50  0001 C CNN
@@
 $EndComp
 $Comp
-L power:GND #PWR061
+L power:GND #PWR059
 U 1 1 5DF7B7C2
 P 5425 4225
-F 0 "#PWR061" H 5425 3975 50  0001 C CNN
+F 0 "#PWR059" H 5425 3975 50  0001 C CNN
 F 1 "GND" H 5430 4052 50  0000 C CNN
 F 2 "" H 5425 4225 50  0001 C CNN
@@
 $EndComp
 $Comp
-L power:+3V3 #PWR057
+L power:+3V3 #PWR055
 U 1 1 5DF7BDF6
 P 5225 2525
-F 0 "#PWR057" H 5225 2375 50  0001 C CNN
+F 0 "#PWR055" H 5225 2375 50  0001 C CNN
 F 1 "+3V3" H 5240 2698 50  0000 C CNN
 F 2 "" H 5225 2525 50  0001 C CNN
@@
 	5425 2525 5425 2825
 $Comp
-L power:GND #PWR058
+L power:GND #PWR056
 U 1 1 5DF80C9B
 P 5725 2525
-F 0 "#PWR058" H 5725 2275 50  0001 C CNN
+F 0 "#PWR056" H 5725 2275 50  0001 C CNN
 F 1 "GND" H 5730 2352 50  0000 C CNN
 F 2 "" H 5725 2525 50  0001 C CNN
@@
 $EndComp
 $Comp
-L power:+3V3 #PWR063
+L power:+3V3 #PWR061
 U 1 1 5DF854B1
 P 5075 5100
-F 0 "#PWR063" H 5075 4950 50  0001 C CNN
+F 0 "#PWR061" H 5075 4950 50  0001 C CNN
 F 1 "+3V3" H 5090 5273 50  0000 C CNN
 F 2 "" H 5075 5100 50  0001 C CNN
