File: Hardware/Motor_Control_PCB/KiCAD_Project/motor_control/Power.sch (KiCad schematic (older format))
At the start: 10 parts, among them J7 Battery, J8 External Power Switch, U3 LT1521-3.3

Commit message: Update part numbers. Motor control Rev 1.0 complete.
Parts:
- C10, C13: Internal Part Number 1-0000075 -> 1-0000005
Changed lines of the file:
@@
 F 2 "Capacitors_SMD:C_0603_HandSoldering" H 4463 3225 50  0001 C CNN
 F 3 "~" H 4425 3375 50  0001 C CNN
-F 4 "1-0000075" H 4425 3375 50  0001 C CNN "Internal Part Number"
+F 4 "1-0000005" H 4425 3375 50  0001 C CNN "Internal Part Number"
 F 5 "1" H 4425 3375 50  0001 C CNN "Populated"
 	1    4425 3375
@@
 F 2 "Capacitors_SMD:C_0603_HandSoldering" H 6563 3225 50  0001 C CNN
 F 3 "~" H 6525 3375 50  0001 C CNN
-F 4 "1-0000075" H 6525 3375 50  0001 C CNN "Internal Part Number"
+F 4 "1-0000005" H 6525 3375 50  0001 C CNN "Internal Part Number"
 F 5 "1" H 6525 3375 50  0001 C CNN "Populated"
 	1    6525 3375
