File: Hardware/Motor_Control_PCB/KiCAD_Project/motor_control/motor_control.kicad_pcb (KiCad board)
At the start: 4 copper layers, 58.4 x 45.7 mm, 57 parts, among them J1 Motor, J2 Conn_01x02, J3 ISP, J4 Spares 2, J5 Spares 1, J6 UART1, J7 Battery, J8 External Power Switch, Q1 MMBT3904, SW1 Configuration, U1 INA169, U2 STM32F103CBT6, U3 LT1521-3.3, Y1 8MHz

Commit message: Update BOM and misc. metadata
Parts:
- added PCB1: barepcb, lib_fp:barepcb, F.Cu at (117.6, 75.2)
