File: Hardware/Battery_PCB/KiCAD_Project/battery_pack/battery_pack.kicad_pcb (KiCad board)
At the start: 2 copper layers, 91.4 x 43.2 mm, 9 parts, among them J1 Conn_01x02

Commit message: Update metadata and BOM
Parts:
- added PCB1: barepcb, lib_fp:barepcb, F.Cu at (72.1, 16.5)
Changed lines of the file:
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@@
-(kicad_pcb (version 20171130) (host pcbnew "(5.1.4)-1")
+(kicad_pcb (version 20171130) (host pcbnew "(5.1.7)-1")
   (general
     (thickness 1.6)
@@
     (tracks 17)
     (zones 0)
-    (modules 9)
+    (modules 10)
     (nets 6)
   )
   (page A4)
+  (title_block
+    (title "Battery Pack - NSSL EFM")
+    (date 2020-12-18)
+    (rev 1.0)
+    (company "Leeman Geophysical LLC")
+    (comment 1 "(479) 373-3736")
+    (comment 2 "Siloam Springs, AR 72761")
+    (comment 3 "850 South Lincoln St.")
+  )
   (layers
     (0 F.Cu signal hide)
@@
       (effects (font (size 1 1) (thickness 0.15)))
     )
+    (fp_line (start -19 9) (end -19 -9) (layer F.SilkS) (width 0.15))
+    (fp_line (start 19 9) (end -19 9) (layer F.SilkS) (width 0.15))
+    (fp_line (start 19 -9) (end 19 9) (layer F.SilkS) (width 0.15))
     (fp_line (start -19 -9) (end 19 -9) (layer F.SilkS) (width 0.15))
-    (fp_line (start 19 -9) (end 19 9) (layer F.SilkS) (width 0.15))
-    (fp_line (start 19 9) (end -19 9) (layer F.SilkS) (width 0.15))
-    (fp_line (start -19 9) (end -19 -9) (layer F.SilkS) (width 0.15))
     (pad 2 thru_hole circle (at -15.695 0 90) (size 1.87 1.87) (drill 1.17) (layers *.Cu *.Mask)
       (net 1 "Net-(BT1-Pad2)"))
@@
       (effects (font (size 1 1) (thickness 0.15)))
     )
+    (fp_line (start -19 -9) (end 19 -9) (layer F.SilkS) (width 0.15))
+    (fp_line (start 19 -9) (end 19 9) (layer F.SilkS) (width 0.15))
+    (fp_line (start 19 9) (end -19 9) (layer F.SilkS) (width 0.15))
     (fp_line (start -19 9) (end -19 -9) (layer F.SilkS) (width 0.15))
-    (fp_line (start 19 9) (end -19 9) (layer F.SilkS) (width 0.15))
-    (fp_line (start 19 -9) (end 19 9) (layer F.SilkS) (width 0.15))
-    (fp_line (start -19 -9) (end 19 -9) (layer F.SilkS) (width 0.15))
     (pad "" np_thru_hole circle (at 15.695 7.11 270) (size 2.36 2.36) (drill 2.36) (layers *.Cu *.Mask))
     (pad "" np_thru_hole circle (at 8.66 0 270) (size 3.18 3.18) (drill 3.18) (layers *.Cu *.Mask))
@@
       (effects (font (size 1 1) (thickness 0.15)))
     )
+    (fp_line (start -19 -9) (end 19 -9) (layer F.SilkS) (width 0.15))
+    (fp_line (start 19 -9) (end 19 9) (layer F.SilkS) (width 0.15))
+    (fp_line (start 19 9) (end -19 9) (layer F.SilkS) (width 0.15))
     (fp_line (start -19 9) (end -19 -9) (layer F.SilkS) (width 0.15))
-    (fp_line (start 19 9) (end -19 9) (layer F.SilkS) (width 0.15))
-    (fp_line (start 19 -9) (end 19 9) (layer F.SilkS) (width 0.15))
-    (fp_line (start -19 -9) (end 19 -9) (layer F.SilkS) (width 0.15))
     (pad "" np_thru_hole circle (at 15.695 7.11 90) (size 2.36 2.36) (drill 2.36) (layers *.Cu *.Mask))
     (pad "" np_thru_hole circle (at 8.66 0 90) (size 3.18 3.18) (drill 3.18) (layers *.Cu *.Mask))
@@
       (effects (font (size 1 1) (thickness 0.15)))
     )
+    (fp_line (start -19 9) (end -19 -9) (layer F.SilkS) (width 0.15))
+    (fp_line (start 19 9) (end -19 9) (layer F.SilkS) (width 0.15))
+    (fp_line (start 19 -9) (end 19 9) (layer F.SilkS) (width 0.15))
     (fp_line (start -19 -9) (end 19 -9) (layer F.SilkS) (width 0.15))
-    (fp_line (start 19 -9) (end 19 9) (layer F.SilkS) (width 0.15))
-    (fp_line (start 19 9) (end -19 9) (layer F.SilkS) (width 0.15))
-    (fp_line (start -19 9) (end -19 -9) (layer F.SilkS) (width 0.15))
     (pad 2 thru_hole circle (at -15.695 0 270) (size 1.87 1.87) (drill 1.17) (layers *.Cu *.Mask)
       (net 5 "Net-(BT4-Pad2)"))
@@
       (effects (font (size 1 1) (thickness 0.15)))
     )
+    (fp_circle (center 0 0) (end 2.85 0) (layer Cmts.User) (width 0.15))
     (fp_circle (center 0 0) (end 3.1 0) (layer F.CrtYd) (width 0.05))
-    (fp_circle (center 0 0) (end 2.85 0) (layer Cmts.User) (width 0.15))
     (fp_text user %R (at 0.3 0) (layer F.Fab)
       (effects (font (size 1 1) (thickness 0.15)))
@@
       (effects (font (size 1 1) (thickness 0.15)))
     )
+    (fp_circle (center 0 0) (end 3.1 0) (layer F.CrtYd) (width 0.05))
+    (fp_circle (center 0 0) (end 2.85 0) (layer Cmts.User) (width 0.15))
     (fp_text user %R (at 0.3 0) (layer F.Fab)
       (effects (font (size 1 1) (thickness 0.15)))
     )
-    (fp_circle (center 0 0) (end 2.85 0) (layer Cmts.User) (width 0.15))
-    (fp_circle (center 0 0) (end 3.1 0) (layer F.CrtYd) (width 0.05))
     (pad 1 np_thru_hole circle (at 0 0) (size 3.2 3.2) (drill 3.2) (layers *.Cu *.Mask))
   )
@@
       (effects (font (size 1 1) (thickness 0.15)))
     )
+    (fp_circle (center 0 0) (end 2.85 0) (layer Cmts.User) (width 0.15))
     (fp_circle (center 0 0) (end 3.1 0) (layer F.CrtYd) (width 0.05))
-    (fp_circle (center 0 0) (end 2.85 0) (layer Cmts.User) (width 0.15))
     (fp_text user %R (at 0.3 0) (layer F.Fab)
       (effects (font (size 1 1) (thickness 0.15)))
@@
       (effects (font (size 1 1) (thickness 0.15)))
     )
+    (fp_circle (center 0 0) (end 3.1 0) (layer F.CrtYd) (width 0.05))
+    (fp_circle (center 0 0) (end 2.85 0) (layer Cmts.User) (width 0.15))
     (fp_text user %R (at 0.3 0) (layer F.Fab)
       (effects (font (size 1 1) (thickness 0.15)))
     )
-    (fp_circle (center 0 0) (end 2.85 0) (layer Cmts.User) (width 0.15))
-    (fp_circle (center 0 0) (end 3.1 0) (layer F.CrtYd) (width 0.05))
     (pad 1 np_thru_hole circle (at 0 0) (size 3.2 3.2) (drill 3.2) (layers *.Cu *.Mask))
   )
@@
       (effects (font (size 1 1) (thickness 0.15)))
     )
+    (fp_line (start -0.635 -1.27) (end 1.27 -1.27) (layer F.Fab) (width 0.1))
+    (fp_line (start 1.27 -1.27) (end 1.27 3.81) (layer F.Fab) (width 0.1))
+    (fp_line (start 1.27 3.81) (end -1.27 3.81) (layer F.Fab) (width 0.1))
+    (fp_line (start -1.27 3.81) (end -1.27 -0.635) (layer F.Fab) (width 0.1))
+    (fp_line (start -1.27 -0.635) (end -0.635 -1.27) (layer F.Fab) (width 0.1))
+    (fp_line (start -1.33 3.87) (end 1.33 3.87) (layer F.SilkS) (width 0.12))
+    (fp_line (start -1.33 1.27) (end -1.33 3.87) (layer F.SilkS) (width 0.12))
+    (fp_line (start 1.33 1.27) (end 1.33 3.87) (layer F.SilkS) (width 0.12))
+    (fp_line (start -1.33 1.27) (end 1.33 1.27) (layer F.SilkS) (width 0.12))
+    (fp_line (start -1.33 0) (end -1.33 -1.33) (layer F.SilkS) (width 0.12))
+    (fp_line (start -1.33 -1.33) (end 0 -1.33) (layer F.SilkS) (width 0.12))
+    (fp_line (start -1.8 -1.8) (end -1.8 4.35) (layer F.CrtYd) (width 0.05))
+    (fp_line (start -1.8 4.35) (end 1.8 4.35) (layer F.CrtYd) (width 0.05))
+    (fp_line (start 1.8 4.35) (end 1.8 -1.8) (layer F.CrtYd) (width 0.05))
+    (fp_line (start 1.8 -1.8) (end -1.8 -1.8) (layer F.CrtYd) (width 0.05))
     (fp_text user %R (at 0 1.27 90) (layer F.Fab)
       (effects (font (size 1 1) (thickness 0.15)))
     )
-    (fp_line (start 1.8 -1.8) (end -1.8 -1.8) (layer F.CrtYd) (width 0.05))
-    (fp_line (start 1.8 4.35) (end 1.8 -1.8) (layer F.CrtYd) (width 0.05))
-    (fp_line (start -1.8 4.35) (end 1.8 4.35) (layer F.CrtYd) (width 0.05))
-    (fp_line (start -1.8 -1.8) (end -1.8 4.35) (layer F.CrtYd) (width 0.05))
-    (fp_line (start -1.33 -1.33) (end 0 -1.33) (layer F.SilkS) (width 0.12))
-    (fp_line (start -1.33 0) (end -1.33 -1.33) (layer F.SilkS) (width 0.12))
-    (fp_line (start -1.33 1.27) (end 1.33 1.27) (layer F.SilkS) (width 0.12))
-    (fp_line (start 1.33 1.27) (end 1.33 3.87) (layer F.SilkS) (width 0.12))
-    (fp_line (start -1.33 1.27) (end -1.33 3.87) (layer F.SilkS) (width 0.12))
-    (fp_line (start -1.33 3.87) (end 1.33 3.87) (layer F.SilkS) (width 0.12))
-    (fp_line (start -1.27 -0.635) (end -0.635 -1.27) (layer F.Fab) (width 0.1))
-    (fp_line (start -1.27 3.81) (end -1.27 -0.635) (layer F.Fab) (width 0.1))
-    (fp_line (start 1.27 3.81) (end -1.27 3.81) (layer F.Fab) (width 0.1))
-    (fp_line (start 1.27 -1.27) (end 1.27 3.81) (layer F.Fab) (width 0.1))
-    (fp_line (start -0.635 -1.27) (end 1.27 -1.27) (layer F.Fab) (width 0.1))
     (pad 2 thru_hole oval (at 0 2.54) (size 1.7 1.7) (drill 1) (layers *.Cu *.Mask)
       (net 5 "Net-(BT4-Pad2)"))
@@
     )
   )
+  (module lib_fp:barepcb (layer F.Cu)
+    (at 72.136 16.51)
+    (fp_text reference PCB1 (at 0 0.5) (layer Dwgs.User)
+      (effects (font (size 1 1) (thickness 0.15)))
+    )
+    (fp_text value barepcb (at 0 -0.5) (layer F.Fab)
+      (effects (font (size 1 1) (thickness 0.15)))
+    )
+    (fp_line (start -3.5 -1.5) (end 3.5 -1.5) (layer F.CrtYd) (width 0.12))
+    (fp_line (start 3.5 -1.5) (end 3.5 1.5) (layer F.CrtYd) (width 0.12))
+    (fp_line (start 3.5 1.5) (end -3.5 1.5) (layer F.CrtYd) (width 0.12))
+    (fp_line (start -3.5 1.5) (end -3.5 -1.5) (layer F.CrtYd) (width 0.12))
+  )
   (gr_text "CR2 Battery Carrier\nRev 1.0 - November 2019\nP/N 3-0000020" (at 114.554 60.706) (layer B.SilkS)
