File: Hardware/Battery_PCB/KiCAD_Project/battery_pack/battery_pack.sch (KiCad schematic (older format))
At the start: 9 parts, among them J1 Conn_01x02

Commit message: Update metadata and BOM
Parts:
- added PCB1: barepcb, lib_fp:barepcb, symbol lib_sch:barepcb
Changed lines of the file:
@@
 EESchema Schematic File Version 4
-LIBS:battery_pack-cache
 EELAYER 30 0
 EELAYER END
@@
 	1    0    0    -1
 $EndComp
+$Comp
+L lib_sch:barepcb PCB1
+U 1 1 5FDCC3D1
+P 7250 6375
+F 0 "PCB1" H 7478 6421 50  0000 L CNN
+F 1 "barepcb" H 7100 6375 50  0000 L CNN
+F 2 "lib_fp:barepcb" H 7250 6375 50  0001 C CNN
+F 3 "" H 7250 6375 50  0001 C CNN
+F 4 "3-0000020" H 7250 6375 50  0001 C CNN "Internal Part Number"
+F 5 "1" H 7250 6375 50  0001 C CNN "Populated"
+	1    7250 6375
+	1    0    0    -1
+$EndComp
