File: Hardware/Tracker_PCB/KiCAD_Project/tracker/tracker.sch (KiCad schematic (older format))
At the start: 58 parts, among them J1 RockBlock9603, J2 Switch, J3 Battery, J4 ICSP, Q1 BSS138, Q2 BSS138, SW1 SW_SPST, U1 XBee, U2 ATmega328P-AU, U3 TSR2, U4 RockBlockMechanical, U5 ublox_SAM-M8Q, U6 MIC5219-3.3YM5, Y1 16MHz

Commit message: Initial layout
Parts:
- J2: value Switch -> Regulator Bypass
Connections:
- wire segments 132 -> 129
Other:
- moved on the sheet: J2
Changed lines of the file:
@@
 L Connector_Generic:Conn_01x02 J2
 U 1 1 5FFB5D23
-P 1425 5500
-F 0 "J2" V 1389 5312 50  0000 R CNN
-F 1 "Switch" V 1298 5312 50  0000 R CNN
-F 2 "" H 1425 5500 50  0001 C CNN
-F 3 "~" H 1425 5500 50  0001 C CNN
-	1    1425 5500
+P 2675 5300
+F 0 "J2" V 2639 5112 50  0000 R CNN
+F 1 "Regulator Bypass" V 2775 5550 50  0000 R CNN
+F 2 "" H 2675 5300 50  0001 C CNN
+F 3 "~" H 2675 5300 50  0001 C CNN
+	1    2675 5300
 	0    -1   -1   0
 $EndComp
-Wire Wire Line
-	1125 6050 1200 6050
-Wire Wire Line
-	1425 5700 1200 5700
-Wire Wire Line
-	1200 5700 1200 6050
-Wire Wire Line
-	1200 6050 1275 6050
-Wire Wire Line
-	1525 5700 1750 5700
-Wire Wire Line
-	1750 5700 1750 6050
-Wire Wire Line
-	1750 6050 1675 6050
 $Comp
 L power:GND #PWR028
@@
 	0    1    1    0
 $EndComp
-Connection ~ 1200 6050
 $Comp
 L capacitors_0603:1-0000007 C10
@@
 	1875 6125 1875 6050
 Wire Wire Line
-	1875 6050 1750 6050
-Connection ~ 1750 6050
-Wire Wire Line
 	1875 6050 2000 6050
 Connection ~ 1875 6050
@@
 P 2325 6050
 F 0 "#FLG0102" H 2325 6125 50  0001 C CNN
-F 1 "PWR_FLAG" V 2325 5825 50  0000 C CNN
+F 1 "PWR_FLAG" V 2325 6350 50  0000 C CNN
 F 2 "" H 2325 6050 50  0001 C CNN
 F 3 "~" H 2325 6050 50  0001 C CNN
 	1    2325 6050
-	1    0    0    -1
+	-1   0    0    1
 $EndComp
 Connection ~ 2325 6050
@@
 	1    0    0    -1
 $EndComp
+Wire Wire Line
+	1125 6050 1275 6050
+Wire Wire Line
+	1675 6050 1875 6050
+$Comp
+L power:+5V #PWR?
+U 1 1 5FDF517E
+P 3300 5500
+F 0 "#PWR?" H 3300 5350 50  0001 C CNN
+F 1 "+5V" H 3315 5673 50  0000 C CNN
+F 2 "" H 3300 5500 50  0001 C CNN
+F 3 "" H 3300 5500 50  0001 C CNN
+	1    3300 5500
+	1    0    0    -1
+$EndComp
+Wire Wire Line
+	3300 5500 2775 5500
+Wire Wire Line
+	2675 5500 2325 5500
+Wire Wire Line
+	2325 5500 2325 6050
 $EndSCHEMATC
