File: Hardware/Tracker_PCB/KiCAD_Project/tracker/tracker.kicad_pcb (KiCad board)
At the start: 2 copper layers, 78.7 x 57.2 mm, 58 parts, among them J1 RockBlock9603, J2 ICSP, J4 Battery, Q1 BSS138, Q2 BSS138, SW1 SW_SPST, U1 XBee, U2 ATmega328P-AU, U3 TSR2, U4 RockBlockMechanical, U5 ublox_SAM-M8Q, U6 MIC5219-3.3YM5, Y1 16MHz

Commit message: Initial Layout
Parts:
- moved C10 8.13 mm to (136.7, 90.2)
- moved C11 1.27 mm to (132.1, 143.3)
- moved R16 1.27 mm to (136.9, 135.9)
- moved C9 1.27 mm to (124.2, 143.3)
- moved U5 1.27 mm to (127.0, 134.1)
- turned F1 to 90 degrees
Routing:
- net RB_5V: track 0.00 -> 85.2 mm, vias 0 -> 4
- net RESET: track 0.00 -> 73.6 mm, vias 0 -> 4
- net RB_GND: track 0.00 -> 57.3 mm, vias 0 -> 27
- net RB_RXI_3V3: track 0.00 -> 50.7 mm, vias 0 -> 4
- net RB_TXO_3V3: track 0.00 -> 47.2 mm, vias 0 -> 2
- net Net-(R14-Pad2): track 0.00 -> 46.5 mm, vias 0 -> 2
- net GPS_PPS: track 0.00 -> 45.8 mm, vias 0 -> 2
- net +3V3: track 0.00 -> 44.2 mm, vias 0 -> 14
- net Net-(R15-Pad2): track 0.00 -> 38.0 mm, vias 0 -> 2
- net RB_NetAv: track 0.00 -> 35.9 mm, vias 0 -> 3
- net Net-(R12-Pad2): track 0.00 -> 32.7 mm, vias 0 -> 2
- net Net-(R13-Pad2): track 0.00 -> 31.2 mm, vias 0 -> 2
- net Net-(BT1-Pad1): track 0.00 -> 27.7 mm
- net Net-(F1-Pad1): track 0.00 -> 21.7 mm
- net Net-(R9-Pad1): track 0.00 -> 20.5 mm
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- added copper zone on In1.Cu, net +3V3
- added copper zone on In2.Cu, net RB_GND
Other:
- copper layers 2 -> 4
- net class Default: clearance 0.2 -> 0.1524; trace_width 0.25 -> 0.1524; via_dia 0.8 -> 0.508; via_drill 0.4 -> 0.254
- rule trace_clearance: 0.2 -> 0.1524
- rule trace_min: 0.2 -> 0.1524
- rule via_min_drill: 0.3 -> 0.254
- rule via_min_size: 0.4 -> 0.508
- board text added: "ON"

Commit message: Tweak layout and make production files.
Other:
- board text added: "Balloon Tracker/Cutdown Command 3-0000068"
Changed lines of the file:
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@@
   (general
     (thickness 1.6)
-    (drawings 5)
+    (drawings 6)
     (tracks 347)
     (zones 0)
@@
   (title_block
     (title "Balloon Sat Tracker")
-    (date 2020-12-18)
+    (date 2020-12-22)
     (rev 1.0)
     (company "Leeman Geophysical LLC")
@@
   )
   (setup
-    (last_trace_width 0.3048)
+    (last_trace_width 0.1524)
     (user_trace_width 0.1524)
     (user_trace_width 0.3048)
@@
       (outputformat 1)
       (mirror false)
-      (drillshape 1)
+      (drillshape 0)
       (scaleselection 1)
-      (outputdirectory ""))
+      (outputdirectory "../../Production/GERBERS/"))
   )
   (net 0 "")
@@
       (effects (font (size 1 1) (thickness 0.15)))
     )
-    (pad 1 smd roundrect (at -2.1375 0 90) (size 1.125 3.4) (layers F.Cu F.Paste F.Mask) (roundrect_rratio 0.222222)
+    (pad 1 smd roundrect (at -2.1375 0 90) (size 1.125 3.4) (layers F.Cu F.Paste F.Mask) (roundrect_rratio 0.2222213333333333)
       (net 13 "Net-(F1-Pad1)"))
-    (pad 2 smd roundrect (at 2.1375 0 90) (size 1.125 3.4) (layers F.Cu F.Paste F.Mask) (roundrect_rratio 0.222222)
+    (pad 2 smd roundrect (at 2.1375 0 90) (size 1.125 3.4) (layers F.Cu F.Paste F.Mask) (roundrect_rratio 0.2222213333333333)
       (net 7 "Net-(C10-Pad1)"))
     (model ${KISYS3DMOD}/Fuse.3dshapes/Fuse_1812_4532Metric.wrl
@@
   (module lib_fp:picoblade (layer B.Cu)
     (at 174.752 98.552 90)
-    (fp_text reference J1 (at -2.5 5.5 90) (layer B.SilkS)
+    (fp_text reference J1 (at 0 4.826 90) (layer B.SilkS)
       (effects (font (size 1 1) (thickness 0.15)) (justify mirror))
     )
@@
   (module lib_fp:RockBlock_Mechanical (layer B.Cu)
     (at 139.954 115.824 270)
-    (fp_text reference U4 (at 24.13 -21.59 180) (layer B.SilkS)
+    (fp_text reference U4 (at -23.368 -21.336 180) (layer B.SilkS)
       (effects (font (size 1 1) (thickness 0.15)) (justify mirror))
     )
@@
       (net 38 "Net-(U2-Pad8)"))
   )
+  (gr_text "Balloon Tracker/Cutdown Command\n3-0000068" (at 139.954 141.986) (layer B.SilkS)
+    (effects (font (size 1.5 1.5) (thickness 0.3)) (justify mirror))
+  )
   (gr_text ON (at 120.396 104.394) (layer F.SilkS)
