File: Hardware/Cutdown_PCB/KiCAD_Project/cutdown/cutdown.kicad_pcb (KiCad board)
At the start: 4 copper layers, 24.1 x 60.3 mm, 26 parts, among them J1 Nichrome Wire, Q1 MMBT3904, U1 Particle, U2 BMP388, U3 ublox_SAM-M8Q

Commit message: Initial layout
Parts:
- removed BZ1: Buzzer, lib_fp:PS1240P02BT
- added BT2: CR123, lib_fp:1-0000782, B.Cu at (133.3, 52.1)
- added C10: 1-0000075, capacitors_0805:1-0000075, F.Cu at (107.2, 132.8)
- added C11: 1-0000075, capacitors_0805:1-0000075, F.Cu at (114.8, 136.4)
- added C12: 1-0000018, capacitors_0603:1-0000018, F.Cu at (116.8, 136.4)
- added C13: 1-0000075, capacitors_0805:1-0000075, F.Cu at (118.4, 131.1)
- added C14: 1-0000075, capacitors_0805:1-0000075, F.Cu at (114.0, 155.4)
- added C15: 1-0000018, capacitors_0603:1-0000018, F.Cu at (114.0, 157.5)
- added C16: 1-0000007, capacitors_0603:1-0000007, F.Cu at (114.0, 159.3)
- added C17: 1-0000007, capacitors_0603:1-0000007, F.Cu at (125.2, 171.7)
- added C18: 0.1u, Capacitor_SMD:C_0603_1608Metric, F.Cu at (131.6, 145.3)
- added C19: 0.1u, Capacitor_SMD:C_0603_1608Metric, F.Cu at (131.6, 143.5)
- added C5: 1-0000007, capacitors_0603:1-0000007, F.Cu at (141.0, 131.1)
- added C6: 1-0000007, capacitors_0603:1-0000007, F.Cu at (126.2, 130.0)
- added C7: 1-0000007, capacitors_0603:1-0000007, F.Cu at (126.2, 128.3)
- added C8: 1-0000007, capacitors_0603:1-0000007, F.Cu at (133.6, 121.4)
- added C9: 1-0000007, capacitors_0603:1-0000007, F.Cu at (141.0, 129.3)
- added D1: Green, LED_SMD:LED_0805_2012Metric, F.Cu at (115.8, 114.3)
- added D2: Yellow, LED_SMD:LED_0805_2012Metric, F.Cu at (139.7, 174.2)
- added D3: Red, LED_SMD:LED_0805_2012Metric, F.Cu at (139.7, 172.0)
- added D4: Red, LED_SMD:LED_0805_2012Metric, F.Cu at (111.3, 114.3)
- added D5: Blue, LED_SMD:LED_0805_2012Metric, F.Cu at (109.0, 114.3)
- added D6: Yellow, LED_SMD:LED_0805_2012Metric, F.Cu at (106.7, 114.3)
- added D7: D_Schottky, Diode_SMD:D_SOD-123F, F.Cu at (111.5, 132.8)
- added D8: Yellow, LED_SMD:LED_0805_2012Metric, F.Cu at (113.5, 114.3)
- added J2: Battery LiPO 1S, lib_fp:JST_S2B-PH-SM4-TB(LF)(SN), B.Cu at (112.5, 122.2)
- added J3: ISP, Connector_PinHeader_2.54mm:PinHeader_2x03_P2.54mm_Vertical, F.Cu at (136.4, 137.4)
- added J4: Hot Wire, lib_fp:1-0000783, F.Cu at (106.9, 99.1)
- added J5: External Cutdown, lib_fp:JST_S2B-PH-SM4-TB(LF)(SN), B.Cu at (120.7, 149.6)
- added PCB1: barepcb, lib_fp:barepcb, F.Cu at (278.6, 161.5)
- added Q2: FQP30N06L, Package_TO_SOT_THT:TO-220-3_Horizontal_TabDown, F.Cu at (122.4, 110.7)
- added R16: 10k, Resistor_SMD:R_0603_1608Metric, F.Cu at (131.6, 147.8)
- added R17: 10k, Resistor_SMD:R_0603_1608Metric, F.Cu at (141.0, 134.9)
- added R18: NP, Resistor_SMD:R_0603_1608Metric, F.Cu at (141.0, 136.7)
- added R19: 1-0000006, resistors_0603:1-0000006, F.Cu at (121.9, 171.7)
- added R20: 1-0000008, resistors_0603:1-0000008, F.Cu at (109.0, 117.9)
- added R21: 1-0000008, resistors_0603:1-0000008, F.Cu at (106.7, 117.9)
- added R22: 10k, Resistor_SMD:R_0603_1608Metric, F.Cu at (138.4, 145.3)
- added R23: NP, Resistor_SMD:R_0603_1608Metric, F.Cu at (138.4, 148.8)
- added R24: 1-0000006, resistors_0603:1-0000006, F.Cu at (119.9, 116.6)
- added R25: 1-0000010, resistors_0603:1-0000010, F.Cu at (119.9, 109.5)
- added R26: 10k, Resistor_SMD:R_0603_1608Metric, F.Cu at (138.4, 147.1)
- added R27: 1-0000174, resistors_0603:1-0000174, F.Cu at (107.2, 136.4)
- added R28: 1-0000013, resistors_0603:1-0000013, F.Cu at (113.5, 117.9)
- added R29: 1-0000010, resistors_0603:1-0000010, F.Cu at (112.5, 124.7)
- added SW1: SW_SPST, lib_fp:SW_GF-123-0054, F.Cu at (114.3, 145.0)
- added U4: XBee, lib_fp:XBee, B.Cu at (115.1, 164.3)
- added U5: BMP388, lib_fp:PQFN50P200X200X80-10N, F.Cu at (135.4, 145.5)
- added U6: MCP73831, lib_fp:1-0000793, F.Cu at (115.8, 127.5)
- added Y1: 16MHz, lib_fp:Resonator, F.Cu at (127.0, 134.9)
- BT1: value CR1220 -> CR123; footprint lib_fp:S8411-45R -> lib_fp:1-0000782; moved to B.Cu
- C1, C2: value 0.1u -> 1-0000007; footprint Capacitors_SMD:C_0603_HandSoldering -> capacitors_0603:1-0000007; moved to F.Cu
- C3, C4: value 0.1u -> 1-0000017; footprint Capacitors_SMD:C_0603_HandSoldering -> capacitors_0603:1-0000017; moved to F.Cu
- J1: value Nichrome Wire -> Mini_USB_B; footprint Pin_Headers:Pin_Header_Straight_1x04_Pitch2.54mm -> lib_fp:MiniUSB
- Q1: value MMBT3904 -> 2N7002; footprint TO_SOT_Packages_SMD:SOT-23 -> Package_TO_SOT_SMD:SOT-23; moved to F.Cu
- R1: value 10k -> 1-0000008; footprint Resistor_SMD:R_0603_1608Metric_Pad1.05x0.95mm_HandSolder -> resistors_0603:1-0000008; moved to F.Cu
- R10: value 10k -> 1-0000008; footprint Resistor_SMD:R_0603_1608Metric_Pad1.05x0.95mm_HandSolder -> resistors_0603:1-0000008
- R11: value 1k -> 1-0000008; footprint Resistor_SMD:R_0603_1608Metric_Pad1.05x0.95mm_HandSolder -> resistors_0603:1-0000008; moved to F.Cu
- R12: value 1k -> 1-0000010; footprint Resistor_SMD:R_0603_1608Metric_Pad1.05x0.95mm_HandSolder -> resistors_0603:1-0000010; moved to F.Cu
- R13: footprint Resistor_SMD:R_0603_1608Metric_Pad1.05x0.95mm_HandSolder -> Resistor_SMD:R_0603_1608Metric; moved to F.Cu
- R14: value 0R0 -> 10k; footprint Resistor_SMD:R_0603_1608Metric_Pad1.05x0.95mm_HandSolder -> Resistor_SMD:R_0603_1608Metric; moved to F.Cu
- R15: value 0R0 -> 1-0000008; footprint Resistor_SMD:R_0603_1608Metric_Pad1.05x0.95mm_HandSolder -> resistors_0603:1-0000008; moved to F.Cu
- R2: value 10k -> 1-0000006; footprint Resistor_SMD:R_0603_1608Metric_Pad1.05x0.95mm_HandSolder -> resistors_0603:1-0000006; moved to F.Cu
- R3: value 0R0 -> 1-0000013; footprint Resistor_SMD:R_0603_1608Metric_Pad1.05x0.95mm_HandSolder -> resistors_0603:1-0000013
- R4: value 10k -> 1-0000013; footprint Resistor_SMD:R_0603_1608Metric_Pad1.05x0.95mm_HandSolder -> resistors_0603:1-0000013
- R5: value 10k -> 1-0000010; footprint Resistor_SMD:R_0603_1608Metric_Pad1.05x0.95mm_HandSolder -> resistors_0603:1-0000010
- R6: value 10k -> 1-0000010; footprint Resistor_SMD:R_0603_1608Metric_Pad1.05x0.95mm_HandSolder -> resistors_0603:1-0000010; moved to F.Cu
- R7: value 10k -> 1-0000012; footprint Resistor_SMD:R_0603_1608Metric_Pad1.05x0.95mm_HandSolder -> resistors_0603:1-0000012; moved to F.Cu
- R8: value NP -> 1-0000012; footprint Resistor_SMD:R_0603_1608Metric_Pad1.05x0.95mm_HandSolder -> resistors_0603:1-0000012; moved to F.Cu
- R9: value NP -> 1-0000006; footprint Resistor_SMD:R_0603_1608Metric_Pad1.05x0.95mm_HandSolder -> resistors_0603:1-0000006
- U1: value Particle -> FT231XS; footprint lib_fp:Particle -> Package_SO:SSOP-20_3.9x8.7mm_P0.635mm; moved to F.Cu
- U2: value BMP388 -> SPX3819M5-L-3-3; footprint lib_fp:PQFN50P200X200X80-10N -> Package_TO_SOT_SMD:SOT-23-5; moved to F.Cu
- U3: value ublox_SAM-M8Q -> ATmega328P-AU; footprint lib_fp:SAM-M8Q -> Package_QFP:TQFP-32_7x7mm_P0.8mm
- moved R7 132.0 mm to (130.8, 164.6), turned to 0 degrees
- moved R5 132.0 mm to (114.0, 168.4)
- moved Q1 132.0 mm to (114.0, 165.6), turned to 90 degrees
- moved R8 129.6 mm to (130.8, 162.8), turned to 0 degrees
- moved R11 124.0 mm to (136.1, 172.0)
- moved R2 116.8 mm to (125.2, 158.2), turned to 90 degrees
- moved R6 116.5 mm to (114.0, 162.8)
- moved R9 114.8 mm to (116.8, 165.6)
- moved C3 114.1 mm to (130.8, 166.4)
- moved U1 112.2 mm to (124.0, 163.6)
- moved C2 110.1 mm to (121.9, 168.9), turned to 270 degrees
- moved R10 109.5 mm to (136.1, 174.2), turned to 180 degrees
- moved C4 105.1 mm to (130.8, 161.0)
- moved R14 103.7 mm to (134.1, 148.6)
- moved C1 101.1 mm to (123.4, 158.2)
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Connections:
- BT1 pad 1: +BATT -> Net-(BT1-Pad1)
- C2 pad 1: GND -> +3V3
- C2 pad 2: +3V3 -> GND
- C3 pad 1: GND -> Net-(C3-Pad1)
- C3 pad 2: +3V3 -> GND
- C4 pad 1: GND -> Net-(C4-Pad1)
- C4 pad 2: +3V3 -> GND
- J1 pad 1: Net-(J1-Pad1) -> +5V
- J1 pad 2: GND -> Net-(C3-Pad1)
- J1 pad 3: EXT_CUTDOWN -> Net-(C4-Pad1)
- J1 pad 4: GND -> (no net)
- Q1 pad 1: Net-(Q1-Pad1) -> +3V3
- Q1 pad 2: GND -> Net-(Q1-Pad2)
- Q1 pad 3: Net-(BZ1-Pad2) -> DTR
- R1 pad 1: +3V3 -> Net-(D1-Pad2)
- R1 pad 2: BMP388_SDO -> +3V3
- R10 pad 1: Net-(R10-Pad1) -> Net-(D2-Pad1)
- R10 pad 2: GND -> Net-(R10-Pad2)
- R11 pad 1: Net-(Q1-Pad1) -> Net-(D3-Pad1)
- R11 pad 2: PIEZO_ELEMENT -> Net-(R11-Pad2)
- R12 pad 2: Net-(BZ1-Pad2) -> RESET
- R13 pad 2: Net-(R13-Pad2) -> BMP388_INT
- R14 pad 1: Net-(R14-Pad1) -> +3V3
- R14 pad 2: GPS_TX -> SDA
- R15 pad 1: Net-(R15-Pad1) -> Net-(D4-Pad2)
- R15 pad 2: GPS_RX -> Net-(R15-Pad2)
- R2 pad 1: +3V3 -> Net-(R2-Pad1)
- R2 pad 2: BMP388_INT -> +3V3
- R3 pad 1: Net-(J1-Pad1) -> RXI
- R3 pad 2: CUTOFF_LOGIC -> Net-(R3-Pad2)
- R4 pad 1: +3V3 -> TXO
- R4 pad 2: SDA -> Net-(R4-Pad2)
- R5 pad 1: +3V3 -> Net-(Q1-Pad2)
- R5 pad 2: SCL -> +3V3
- R6 pad 1: +3V3 -> DTR
- R6 pad 2: GPS_PPS -> +3V3
- R7 pad 1: +3V3 -> Net-(R7-Pad1)
- R7 pad 2: EXT_CUTDOWN -> Net-(C3-Pad1)
- R8 pad 1: GND -> Net-(R8-Pad1)
- R8 pad 2: EXT_CUTDOWN -> Net-(C4-Pad1)
- R9 pad 1: +3V3 -> Net-(Q1-Pad2)
- R9 pad 2: Net-(R10-Pad1) -> DTR
- U1 pad 1: Net-(U1-Pad1) -> Net-(Q1-Pad2)
- U1 pad 10: Net-(U1-Pad10) -> Net-(R11-Pad2)
- U1 pad 11: Net-(U1-Pad11) -> Net-(R8-Pad1)
- U1 pad 12: Net-(U1-Pad12) -> Net-(R7-Pad1)
- U1 pad 13: Net-(U1-Pad13) -> Net-(R2-Pad1)
- U1 pad 14: Net-(R14-Pad1) -> (no net)
- U1 pad 15: Net-(R15-Pad1) -> +3V3
- U1 pad 16: Net-(U1-Pad16) -> GND
- U1 pad 17: Net-(U1-Pad17) -> Net-(R10-Pad2)
- U1 pad 18: Net-(U1-Pad18) -> (no net)
- U1 pad 19: Net-(U1-Pad19) -> (no net)
- U1 pad 2: +3V3 -> (no net)
- U1 pad 20: Net-(U1-Pad20) -> Net-(R3-Pad2)
- U1 pad 3: Net-(U1-Pad3) -> +3V3
- U1 pad 4: GND -> Net-(R4-Pad2)
- U1 pad 5: PIEZO_ELEMENT -> (no net)
- U1 pad 6: Net-(U1-Pad6) -> GND
- U1 pad 7: Net-(U1-Pad7) -> (no net)
- U1 pad 8: Net-(U1-Pad8) -> (no net)
- U1 pad 9: Net-(U1-Pad9) -> (no net)
- U2 pad 1: +3V3 -> Net-(C10-Pad1)
- U2 pad 2: SCL -> GND
- U2 pad 3: GND -> Net-(R27-Pad2)
- U2 pad 4: SDA -> (no net)
- U2 pad 5: Net-(R10-Pad1) -> +3V3
- U3 pad 1: GND -> XBee_from_uC
- U3 pad 10: GND -> Net-(R15-Pad2)
- U3 pad 11: GND -> (no net)
- U3 pad 12: Net-(U3-Pad12) -> EXT_CUTDOWN
- U3 pad 13: GPS_TX -> Cutdown_Command
- U3 pad 14: GPS_RX -> (no net)
- U3 pad 15: GND -> MOSI
- U3 pad 16: GND -> MISO
- U3 pad 17: +3V3 -> SCK
- U3 pad 18: Net-(U3-Pad18) -> +3V3
- U3 pad 19: Net-(U3-Pad19) -> (no net)
- U3 pad 2: +3V3 -> BMP388_INT
- U3 pad 20: GND -> Net-(C9-Pad1)
- U3 pad 3: +BATT -> GND
- U3 pad 4: GND -> +3V3
- U3 pad 6: GND -> +3V3
- U3 pad 7: GPS_PPS -> Net-(U3-Pad7)
- U3 pad 9: Net-(U3-Pad9) -> (no net)
Routing:
- net +5V: track 0.00 -> 100.5 mm, vias 0 -> 2
- net DTR: track 0.00 -> 84.5 mm, vias 0 -> 4
- net Net-(R21-Pad2): track 0.00 -> 75.1 mm, vias 0 -> 2
- net RESET: track 0.00 -> 71.2 mm, vias 0 -> 4
- net Net-(R4-Pad2): track 0.00 -> 60.8 mm, vias 0 -> 4
- net Net-(R3-Pad2): track 0.00 -> 56.4 mm, vias 0 -> 2
- net GND: track 30.3 -> 83.2 mm, vias 16 -> 40
- net Net-(R20-Pad1): track 0.00 -> 50.0 mm, vias 0 -> 2
- net EXT_CUTDOWN: track 89.0 -> 41.4 mm, vias 0 -> 3
- net CUTOFF_LOGIC: track 46.8 -> 0.00 mm, vias 1 -> 0
- net Net-(R15-Pad2): track 0.00 -> 43.6 mm, vias 0 -> 4
- net XBee_to_uC: track 0.00 -> 42.9 mm, vias 0 -> 2
- net Net-(BT2-Pad1): track 0.00 -> 39.5 mm
- net XBee_from_uC: track 0.00 -> 37.0 mm, vias 0 -> 2
- net PIEZO_ELEMENT: track 34.0 -> 0.00 mm, vias 1 -> 0
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Other:
- board size 24.1 x 60.3 mm -> 43.2 x 152.4 mm
- board text added: "Assoc"
- board text added: "BATT"
- board text added: "Charge"
- board text added: "EXT"
- board text added: "Error"
- board text added: "ON"
- board text added: "Power"
- board text added: "RSSI"
- board text removed: "Balloon Cutdown Module Rev. 2.0 April 2020 P/N 3-0000028"
- board text removed: "Cut"
- board text removed: "Ext"

Commit message: Tweak schematic and PCB
Parts:
- added FID1: Fiducial, Fiducial:Fiducial_1mm_Mask2mm, F.Cu at (143.5, 26.9)
- added FID2: Fiducial, Fiducial:Fiducial_1mm_Mask2mm, F.Cu at (103.9, 175.8)
- moved J3 40.6 mm to (129.3, 110.0), turned to 180 degrees
- moved J1 2.54 mm to (141.2, 163.8)
- renumbered D7 to D4, D8 to D5, D4 to D6, D5 to D7, D6 to D8, J5 to J3, J3 to J4, J4 to J5, R27 to R13, R28 to R14, R29 to R15, R13 to R16, R14 to R17, R15 to R18, R16 to R19, R17 to R20, R18 to R21, R19 to R22, R20 to R23, R21 to R24, R22 to R25, R23 to R26, R24 to R27, R25 to R28, R26 to R29, U6 to U4, U4 to U5, U5 to U6
Routing:
- net RESET: track 71.2 -> 82.9 mm, vias 4 -> 6
- net EXT_CUTDOWN: track 41.4 -> 52.6 mm
- net Net-(C3-Pad1): track 4.54 -> 7.34 mm
- net Net-(C4-Pad1): track 4.94 -> 7.48 mm
- net +5V: track 100.5 -> 103.0 mm
- net GND: track 83.2 -> 80.7 mm
Other:
- outline, holes or cut-outs redrawn
- board text added: "Balloon Cutdown Rev 3.0 3-0000070"
- board text added: "ID"
