File: Hardware/Cutdown_PCB/KiCAD_Project/cutdown/peripherals.sch (KiCad schematic (older format))
At the start: 12 parts, among them U2 BMP388

Commit message: Initial layout
Parts:
- BT1, BT2: renamed from BT?; footprint (none) -> lib_fp:1-0000782
- C18: renamed from C1; footprint Capacitors_SMD:C_0603_HandSoldering -> Capacitor_SMD:C_0603_1608Metric
- C19: renamed from C2; footprint Capacitors_SMD:C_0603_HandSoldering -> Capacitor_SMD:C_0603_1608Metric
- J4: renamed from J?; footprint (none) -> lib_fp:1-0000783
- Q2: renamed from Q?; footprint Package_DirectFET:DirectFET_ST -> Package_TO_SOT_THT:TO-220-3_Horizontal_TabDown
- R22: renamed from R13; footprint Resistor_SMD:R_0603_1608Metric_Pad1.05x0.95mm_HandSolder -> Resistor_SMD:R_0603_1608Metric
- R23: renamed from R9; footprint Resistor_SMD:R_0603_1608Metric_Pad1.05x0.95mm_HandSolder -> Resistor_SMD:R_0603_1608Metric
- R26: renamed from R10; footprint Resistor_SMD:R_0603_1608Metric_Pad1.05x0.95mm_HandSolder -> Resistor_SMD:R_0603_1608Metric
- gave numbers to parts that had none: 2
- renumbered U2 to U5
Changed lines of the file:
@@
 Sheet 2 2
 Title "Cutdown Module - NSSL EFM"
-Date "2020-03-30"
-Rev "2.0"
+Date "2020-12-18"
+Rev "3.0"
 Comp "Leeman Geophysical LLC"
 Comment1 "(479) 373-3736"
@@
 $EndDescr
 $Comp
-L lib_sch:BMP388 U2
+L lib_sch:BMP388 U5
 U 1 1 5DE9BB3A
 P 3900 2450
-F 0 "U2" H 4175 2800 50  0000 L CNN
+F 0 "U5" H 4175 2800 50  0000 L CNN
 F 1 "BMP388" H 4075 2100 50  0000 L CNN
 F 2 "lib_fp:PQFN50P200X200X80-10N" H 3200 2500 50  0001 C CNN
@@
 $EndComp
 $Comp
-L power:+3V3 #PWR0103
+L power:+3V3 #PWR043
 U 1 1 5DE9BB40
 P 3850 1475
-F 0 "#PWR0103" H 3850 1325 50  0001 C CNN
+F 0 "#PWR043" H 3850 1325 50  0001 C CNN
 F 1 "+3V3" H 3700 1550 50  0000 C CNN
 F 2 "" H 3850 1475 50  0001 C CNN
@@
 $EndComp
 $Comp
-L Device:C C2
+L Device:C C19
 U 1 1 5DE9BB48
 P 4175 1800
-F 0 "C2" V 4125 1900 50  0000 C CNN
+F 0 "C19" V 4125 1900 50  0000 C CNN
 F 1 "0.1u" V 4125 1675 50  0000 C CNN
-F 2 "Capacitors_SMD:C_0603_HandSoldering" H 4213 1650 50  0001 C CNN
+F 2 "Capacitor_SMD:C_0603_1608Metric" H 4213 1650 50  0001 C CNN
 F 3 "~" H 4175 1800 50  0001 C CNN
 F 4 "1-0000007" H 4175 1800 50  0001 C CNN "Internal Part Number"
@@
 $EndComp
 $Comp
-L Device:C C1
+L Device:C C18
 U 1 1 5DE9BB50
 P 3625 1800
-F 0 "C1" V 3575 1675 50  0000 C CNN
+F 0 "C18" V 3575 1675 50  0000 C CNN
 F 1 "0.1u" V 3575 1925 50  0000 C CNN
-F 2 "Capacitors_SMD:C_0603_HandSoldering" H 3663 1650 50  0001 C CNN
+F 2 "Capacitor_SMD:C_0603_1608Metric" H 3663 1650 50  0001 C CNN
 F 3 "~" H 3625 1800 50  0001 C CNN
 F 4 "1-0000007" H 3625 1800 50  0001 C CNN "Internal Part Number"
@@
 Connection ~ 3850 1800
 $Comp
-L power:+3V3 #PWR0104
+L power:+3V3 #PWR044
 U 1 1 5DE9BB5C
 P 3950 1475
-F 0 "#PWR0104" H 3950 1325 50  0001 C CNN
+F 0 "#PWR044" H 3950 1325 50  0001 C CNN
 F 1 "+3V3" H 4100 1550 50  0000 C CNN
 F 2 "" H 3950 1475 50  0001 C CNN
@@
 Connection ~ 3950 1800
 $Comp
-L power:GND #PWR0105
+L power:GND #PWR045
 U 1 1 5DE9BB64
 P 3475 1800
-F 0 "#PWR0105" H 3475 1550 50  0001 C CNN
+F 0 "#PWR045" H 3475 1550 50  0001 C CNN
 F 1 "GND" H 3480 1627 50  0000 C CNN
 F 2 "" H 3475 1800 50  0001 C CNN
@@
 $EndComp
 $Comp
-L power:GND #PWR0106
+L power:GND #PWR046
 U 1 1 5DE9BB6A
 P 4325 1800
-F 0 "#PWR0106" H 4325 1550 50  0001 C CNN
+F 0 "#PWR046" H 4325 1550 50  0001 C CNN
 F 1 "GND" H 4330 1627 50  0000 C CNN
 F 2 "" H 4325 1800 50  0001 C CNN
@@
 SDA
 $Comp
-L power:GND #PWR0107
+L power:GND #PWR052
 U 1 1 5DE9BB73
 P 3900 3050
-F 0 "#PWR0107" H 3900 2800 50  0001 C CNN
+F 0 "#PWR052" H 3900 2800 50  0001 C CNN
 F 1 "GND" H 3905 2877 50  0000 C CNN
 F 2 "" H 3900 3050 50  0001 C CNN
@@
 P 2825 2400
 AR Path="/5DE9BB83" Ref="R?"  Part="1"
-AR Path="/5DE92E14/5DE9BB83" Ref="R9"  Part="1"
-F 0 "R9" V 2725 2350 50  0000 L CNN
+AR Path="/5DE92E14/5DE9BB83" Ref="R23"  Part="1"
+F 0 "R23" V 2725 2350 50  0000 L CNN
 F 1 "NP" V 2825 2350 50  0000 L CNN
-F 2 "Resistor_SMD:R_0603_1608Metric_Pad1.05x0.95mm_HandSolder" V 2755 2400 50  0001 C CNN
+F 2 "Resistor_SMD:R_0603_1608Metric" V 2755 2400 50  0001 C CNN
 F 3 "~" H 2825 2400 50  0001 C CNN
 F 4 "1-0000010" H 2825 2400 50  0001 C CNN "Internal Part Number"
@@
 $EndComp
 $Comp
-L Device:R R10
+L Device:R R26
 U 1 1 5DE9BB8B
 P 2825 2800
-F 0 "R10" V 2725 2750 50  0000 L CNN
+F 0 "R26" V 2725 2750 50  0000 L CNN
 F 1 "10k" V 2825 2725 50  0000 L CNN
-F 2 "Resistor_SMD:R_0603_1608Metric_Pad1.05x0.95mm_HandSolder" V 2755 2800 50  0001 C CNN
+F 2 "Resistor_SMD:R_0603_1608Metric" V 2755 2800 50  0001 C CNN
 F 3 "~" H 2825 2800 50  0001 C CNN
 F 4 "1-0000010" H 2825 2800 50  0001 C CNN "Internal Part Number"
@@
 Connection ~ 2825 2600
 $Comp
-L power:GND #PWR0108
+L power:GND #PWR051
 U 1 1 5DE9BB95
 P 2825 2950
-F 0 "#PWR0108" H 2825 2700 50  0001 C CNN
+F 0 "#PWR051" H 2825 2700 50  0001 C CNN
 F 1 "GND" H 2830 2777 50  0000 C CNN
 F 2 "" H 2825 2950 50  0001 C CNN
@@
 $EndComp
 $Comp
-L power:+3V3 #PWR0109
+L power:+3V3 #PWR048
 U 1 1 5DE9BB9B
 P 2825 2250
-F 0 "#PWR0109" H 2825 2100 50  0001 C CNN
+F 0 "#PWR048" H 2825 2100 50  0001 C CNN
 F 1 "+3V3" H 2840 2423 50  0000 C CNN
 F 2 "" H 2825 2250 50  0001 C CNN
@@
 P 4725 2250
 AR Path="/5DE7F4ED" Ref="R?"  Part="1"
-AR Path="/5DE92E14/5DE7F4ED" Ref="R13"  Part="1"
-F 0 "R13" V 4625 2200 50  0000 L CNN
+AR Path="/5DE92E14/5DE7F4ED" Ref="R22"  Part="1"
+F 0 "R22" V 4625 2200 50  0000 L CNN
 F 1 "10k" V 4725 2175 50  0000 L CNN
-F 2 "Resistor_SMD:R_0603_1608Metric_Pad1.05x0.95mm_HandSolder" V 4655 2250 50  0001 C CNN
+F 2 "Resistor_SMD:R_0603_1608Metric" V 4655 2250 50  0001 C CNN
 F 3 "~" H 4725 2250 50  0001 C CNN
 F 4 "1-0000010" H 4725 2250 50  0001 C CNN "Internal Part Number"
@@
 $EndComp
 $Comp
-L power:+3V3 #PWR0120
+L power:+3V3 #PWR047
 U 1 1 5DE7F4F3
 P 4725 2100
-F 0 "#PWR0120" H 4725 1950 50  0001 C CNN
+F 0 "#PWR047" H 4725 1950 50  0001 C CNN
 F 1 "+3V3" H 4740 2273 50  0000 C CNN
 F 2 "" H 4725 2100 50  0001 C CNN
@@
 	4725 2400 4500 2400
 $Comp
-L Device:Battery_Cell BT?
+L Device:Battery_Cell BT1
 U 1 1 5FDAEB8B
 P 8425 1150
-F 0 "BT?" V 8170 1200 50  0000 C CNN
+F 0 "BT1" V 8170 1200 50  0000 C CNN
 F 1 "CR123" V 8261 1200 50  0000 C CNN
-F 2 "" V 8425 1210 50  0001 C CNN
+F 2 "lib_fp:1-0000782" V 8425 1210 50  0001 C CNN
 F 3 "~" V 8425 1210 50  0001 C CNN
 F 4 "1-0000782" H 8425 1150 50  0001 C CNN "Internal Part Number"
@@
 $EndComp
 $Comp
-L resistors_0603:1-0000006 R?
+L resistors_0603:1-0000006 R24
 U 1 1 5FDB2113
 P 7825 2400
-F 0 "R?" V 7750 2400 50  0000 C CNN
+F 0 "R24" V 7750 2400 50  0000 C CNN
 F 1 "1-0000006" V 7825 2400 50  0001 C CNN
 F 2 "resistors_0603:1-0000006" V 7755 2400 50  0001 C CNN
@@
 $EndComp
 $Comp
-L resistors_0603:1-0000010 R?
+L resistors_0603:1-0000010 R25
 U 1 1 5FDB2B0F
 P 8050 2625
-F 0 "R?" V 8125 2575 50  0000 L CNN
+F 0 "R25" V 8125 2575 50  0000 L CNN
 F 1 "1-0000010" V 8050 2625 50  0001 C CNN
 F 2 "resistors_0603:1-0000010" V 7980 2625 50  0001 C CNN
@@
 $EndComp
 $Comp
-L lib_sch:FQP30N06L Q?
+L lib_sch:FQP30N06L Q2
 U 1 1 5FDB4039
 P 8325 2400
-F 0 "Q?" H 8531 2446 50  0000 L CNN
+F 0 "Q2" H 8531 2446 50  0000 L CNN
 F 1 "FQP30N06L" H 8531 2355 50  0000 L CNN
-F 2 "Package_DirectFET:DirectFET_ST" H 8325 2400 50  0001 C CIN
+F 2 "Package_TO_SOT_THT:TO-220-3_Horizontal_TabDown" H 8325 2400 50  0001 C CIN
 F 3 "https://www.infineon.com/dgdl/Infineon-BSF450NE7NH3-DS-v02_02-EN.pdf?fileId=db3a30433a047ba0013a687e2ae403da" H 8325 2400 50  0001 L CNN
 	1    8325 2400
@@
 $EndComp
 $Comp
-L power:GND #PWR?
+L power:GND #PWR049
 U 1 1 5FDB4AF1
 P 8425 2600
-F 0 "#PWR?" H 8425 2350 50  0001 C CNN
+F 0 "#PWR049" H 8425 2350 50  0001 C CNN
 F 1 "GND" H 8425 2450 50  0000 C CNN
 F 2 "" H 8425 2600 50  0001 C CNN
@@
 	8050 2400 8125 2400
 $Comp
-L power:GND #PWR?
+L power:GND #PWR050
 U 1 1 5FDB62BA
 P 8050 2775
-F 0 "#PWR?" H 8050 2525 50  0001 C CNN
+F 0 "#PWR050" H 8050 2525 50  0001 C CNN
 F 1 "GND" H 8050 2625 50  0000 C CNN
 F 2 "" H 8050 2775 50  0001 C CNN
@@
 $EndComp
 $Comp
-L Connector_Generic:Conn_01x02 J?
+L Connector_Generic:Conn_01x02 J4
 U 1 1 5FDB68FF
 P 8625 1925
-F 0 "J?" H 8705 1917 50  0000 L CNN
+F 0 "J4" H 8705 1917 50  0000 L CNN
 F 1 "Hot Wire" H 8705 1826 50  0000 L CNN
-F 2 "" H 8625 1925 50  0001 C CNN
+F 2 "lib_fp:1-0000783" H 8625 1925 50  0001 C CNN
 F 3 "~" H 8625 1925 50  0001 C CNN
 F 4 "1-0000783" H 8625 1925 50  0001 C CNN "Internal Part Number"
@@
 Cutdown_Command
 $Comp
-L Device:Battery_Cell BT?
+L Device:Battery_Cell BT2
 U 1 1 5FE233BE
 P 8425 1450
-F 0 "BT?" V 8170 1500 50  0000 C CNN
+F 0 "BT2" V 8170 1500 50  0000 C CNN
 F 1 "CR123" V 8261 1500 50  0000 C CNN
-F 2 "" V 8425 1510 50  0001 C CNN
+F 2 "lib_fp:1-0000782" V 8425 1510 50  0001 C CNN
 F 3 "~" V 8425 1510 50  0001 C CNN
 F 4 "1-0000782" H 8425 1450 50  0001 C CNN "Internal Part Number"
@@
 $EndComp
 $Comp
-L power:GND #PWR?
+L power:GND #PWR042
 U 1 1 5FE23F21
 P 8150 1050
-F 0 "#PWR?" H 8150 800 50  0001 C CNN
+F 0 "#PWR042" H 8150 800 50  0001 C CNN
 F 1 "GND" H 8150 900 50  0000 C CNN
 F 2 "" H 8150 1050 50  0001 C CNN

Commit message: Tweak schematic and PCB
Parts:
- Q2: Internal Part Number (none) -> 1-0000449; Populated (none) -> 1
- renumbered J4 to J5, R22 to R25, R23 to R26, R24 to R27, R25 to R28, R26 to R29, U5 to U6
Changed lines of the file:
@@
 Sheet 2 2
 Title "Cutdown Module - NSSL EFM"
-Date "2020-12-18"
+Date "2020-12-22"
 Rev "3.0"
 Comp "Leeman Geophysical LLC"
@@
 $EndDescr
 $Comp
-L lib_sch:BMP388 U5
+L lib_sch:BMP388 U6
 U 1 1 5DE9BB3A
 P 3900 2450
-F 0 "U5" H 4175 2800 50  0000 L CNN
+F 0 "U6" H 4175 2800 50  0000 L CNN
 F 1 "BMP388" H 4075 2100 50  0000 L CNN
 F 2 "lib_fp:PQFN50P200X200X80-10N" H 3200 2500 50  0001 C CNN
@@
 $EndComp
 $Comp
-L power:+3V3 #PWR043
+L power:+3V3 #PWR048
 U 1 1 5DE9BB40
 P 3850 1475
-F 0 "#PWR043" H 3850 1325 50  0001 C CNN
+F 0 "#PWR048" H 3850 1325 50  0001 C CNN
 F 1 "+3V3" H 3700 1550 50  0000 C CNN
 F 2 "" H 3850 1475 50  0001 C CNN
@@
 U 1 1 5DE9BB48
 P 4175 1800
-F 0 "C19" V 4125 1900 50  0000 C CNN
-F 1 "0.1u" V 4125 1675 50  0000 C CNN
+F 0 "C19" V 3975 1800 50  0000 C CNN
+F 1 "0.1u" V 4050 1800 50  0000 C CNN
 F 2 "Capacitor_SMD:C_0603_1608Metric" H 4213 1650 50  0001 C CNN
 F 3 "~" H 4175 1800 50  0001 C CNN
@@
 U 1 1 5DE9BB50
 P 3625 1800
-F 0 "C18" V 3575 1675 50  0000 C CNN
-F 1 "0.1u" V 3575 1925 50  0000 C CNN
+F 0 "C18" V 3425 1800 50  0000 C CNN
+F 1 "0.1u" V 3500 1800 50  0000 C CNN
 F 2 "Capacitor_SMD:C_0603_1608Metric" H 3663 1650 50  0001 C CNN
 F 3 "~" H 3625 1800 50  0001 C CNN
@@
 Connection ~ 3850 1800
 $Comp
-L power:+3V3 #PWR044
+L power:+3V3 #PWR049
 U 1 1 5DE9BB5C
 P 3950 1475
-F 0 "#PWR044" H 3950 1325 50  0001 C CNN
+F 0 "#PWR049" H 3950 1325 50  0001 C CNN
 F 1 "+3V3" H 4100 1550 50  0000 C CNN
 F 2 "" H 3950 1475 50  0001 C CNN
@@
 Connection ~ 3950 1800
 $Comp
-L power:GND #PWR045
+L power:GND #PWR050
 U 1 1 5DE9BB64
 P 3475 1800
-F 0 "#PWR045" H 3475 1550 50  0001 C CNN
+F 0 "#PWR050" H 3475 1550 50  0001 C CNN
 F 1 "GND" H 3480 1627 50  0000 C CNN
 F 2 "" H 3475 1800 50  0001 C CNN
@@
 $EndComp
 $Comp
-L power:GND #PWR046
+L power:GND #PWR051
 U 1 1 5DE9BB6A
 P 4325 1800
-F 0 "#PWR046" H 4325 1550 50  0001 C CNN
+F 0 "#PWR051" H 4325 1550 50  0001 C CNN
 F 1 "GND" H 4330 1627 50  0000 C CNN
 F 2 "" H 4325 1800 50  0001 C CNN
@@
 SDA
 $Comp
-L power:GND #PWR052
+L power:GND #PWR057
 U 1 1 5DE9BB73
 P 3900 3050
-F 0 "#PWR052" H 3900 2800 50  0001 C CNN
+F 0 "#PWR057" H 3900 2800 50  0001 C CNN
 F 1 "GND" H 3905 2877 50  0000 C CNN
 F 2 "" H 3900 3050 50  0001 C CNN
@@
 P 2825 2400
 AR Path="/5DE9BB83" Ref="R?"  Part="1"
-AR Path="/5DE92E14/5DE9BB83" Ref="R23"  Part="1"
-F 0 "R23" V 2725 2350 50  0000 L CNN
+AR Path="/5DE92E14/5DE9BB83" Ref="R26"  Part="1"
+F 0 "R26" V 2725 2350 50  0000 L CNN
 F 1 "NP" V 2825 2350 50  0000 L CNN
 F 2 "Resistor_SMD:R_0603_1608Metric" V 2755 2400 50  0001 C CNN
@@
 $EndComp
 $Comp
-L Device:R R26
+L Device:R R29
 U 1 1 5DE9BB8B
 P 2825 2800
-F 0 "R26" V 2725 2750 50  0000 L CNN
+F 0 "R29" V 2725 2750 50  0000 L CNN
 F 1 "10k" V 2825 2725 50  0000 L CNN
 F 2 "Resistor_SMD:R_0603_1608Metric" V 2755 2800 50  0001 C CNN
@@
 Connection ~ 2825 2600
 $Comp
-L power:GND #PWR051
+L power:GND #PWR056
 U 1 1 5DE9BB95
 P 2825 2950
-F 0 "#PWR051" H 2825 2700 50  0001 C CNN
+F 0 "#PWR056" H 2825 2700 50  0001 C CNN
 F 1 "GND" H 2830 2777 50  0000 C CNN
 F 2 "" H 2825 2950 50  0001 C CNN
@@
 $EndComp
 $Comp
-L power:+3V3 #PWR048
+L power:+3V3 #PWR053
 U 1 1 5DE9BB9B
 P 2825 2250
-F 0 "#PWR048" H 2825 2100 50  0001 C CNN
+F 0 "#PWR053" H 2825 2100 50  0001 C CNN
 F 1 "+3V3" H 2840 2423 50  0000 C CNN
 F 2 "" H 2825 2250 50  0001 C CNN
@@
 P 4725 2250
 AR Path="/5DE7F4ED" Ref="R?"  Part="1"
-AR Path="/5DE92E14/5DE7F4ED" Ref="R22"  Part="1"
-F 0 "R22" V 4625 2200 50  0000 L CNN
+AR Path="/5DE92E14/5DE7F4ED" Ref="R25"  Part="1"
+F 0 "R25" V 4625 2200 50  0000 L CNN
 F 1 "10k" V 4725 2175 50  0000 L CNN
 F 2 "Resistor_SMD:R_0603_1608Metric" V 4655 2250 50  0001 C CNN
@@
 $EndComp
 $Comp
-L power:+3V3 #PWR047
+L power:+3V3 #PWR052
 U 1 1 5DE7F4F3
 P 4725 2100
-F 0 "#PWR047" H 4725 1950 50  0001 C CNN
+F 0 "#PWR052" H 4725 1950 50  0001 C CNN
 F 1 "+3V3" H 4740 2273 50  0000 C CNN
 F 2 "" H 4725 2100 50  0001 C CNN
@@
 $EndComp
 $Comp
-L resistors_0603:1-0000006 R24
+L resistors_0603:1-0000006 R27
 U 1 1 5FDB2113
 P 7825 2400
-F 0 "R24" V 7750 2400 50  0000 C CNN
+F 0 "R27" V 7750 2400 50  0000 C CNN
 F 1 "1-0000006" V 7825 2400 50  0001 C CNN
 F 2 "resistors_0603:1-0000006" V 7755 2400 50  0001 C CNN
@@
 $EndComp
 $Comp
-L resistors_0603:1-0000010 R25
+L resistors_0603:1-0000010 R28
 U 1 1 5FDB2B0F
 P 8050 2625
-F 0 "R25" V 8125 2575 50  0000 L CNN
+F 0 "R28" V 8125 2575 50  0000 L CNN
 F 1 "1-0000010" V 8050 2625 50  0001 C CNN
 F 2 "resistors_0603:1-0000010" V 7980 2625 50  0001 C CNN
@@
 F 2 "Package_TO_SOT_THT:TO-220-3_Horizontal_TabDown" H 8325 2400 50  0001 C CIN
 F 3 "https://www.infineon.com/dgdl/Infineon-BSF450NE7NH3-DS-v02_02-EN.pdf?fileId=db3a30433a047ba0013a687e2ae403da" H 8325 2400 50  0001 L CNN
+F 4 "1-0000449" H 8325 2400 50  0001 C CNN "Internal Part Number"
+F 5 "1" H 8325 2400 50  0001 C CNN "Populated"
 	1    8325 2400
 	1    0    0    -1
 $EndComp
 $Comp
-L power:GND #PWR049
+L power:GND #PWR054
 U 1 1 5FDB4AF1
 P 8425 2600
-F 0 "#PWR049" H 8425 2350 50  0001 C CNN
+F 0 "#PWR054" H 8425 2350 50  0001 C CNN
 F 1 "GND" H 8425 2450 50  0000 C CNN
 F 2 "" H 8425 2600 50  0001 C CNN
@@
 	8050 2400 8125 2400
 $Comp
-L power:GND #PWR050
+L power:GND #PWR055
 U 1 1 5FDB62BA
 P 8050 2775
-F 0 "#PWR050" H 8050 2525 50  0001 C CNN
+F 0 "#PWR055" H 8050 2525 50  0001 C CNN
 F 1 "GND" H 8050 2625 50  0000 C CNN
 F 2 "" H 8050 2775 50  0001 C CNN
@@
 $EndComp
 $Comp
-L Connector_Generic:Conn_01x02 J4
+L Connector_Generic:Conn_01x02 J5
 U 1 1 5FDB68FF
 P 8625 1925
-F 0 "J4" H 8705 1917 50  0000 L CNN
+F 0 "J5" H 8705 1917 50  0000 L CNN
 F 1 "Hot Wire" H 8705 1826 50  0000 L CNN
 F 2 "lib_fp:1-0000783" H 8625 1925 50  0001 C CNN
@@
 $EndComp
 $Comp
-L power:GND #PWR042
+L power:GND #PWR047
 U 1 1 5FE23F21
 P 8150 1050
-F 0 "#PWR042" H 8150 800 50  0001 C CNN
+F 0 "#PWR047" H 8150 800 50  0001 C CNN
 F 1 "GND" H 8150 900 50  0000 C CNN
 F 2 "" H 8150 1050 50  0001 C CNN
