File: Hardware/Cutdown_PCB/KiCAD_Project/cutdown/peripherals.sch (KiCad schematic (older format))
At the start: 10 parts, among them J5 Hot Wire, Q2 FQP30N06L, U6 BMP388

Commit message: Reannotate
Parts:
- renumbered C18 to C17, C19 to C18, J5 to J4, R25 to R24, R26 to R25, R27 to R26, R28 to R27, R29 to R28, U6 to U5
Changed lines of the file:
@@
 $EndDescr
 $Comp
-L lib_sch:BMP388 U6
+L lib_sch:BMP388 U5
 U 1 1 5DE9BB3A
 P 3900 2450
-F 0 "U6" H 4175 2800 50  0000 L CNN
+F 0 "U5" H 4175 2800 50  0000 L CNN
 F 1 "BMP388" H 4075 2100 50  0000 L CNN
 F 2 "lib_fp:PQFN50P200X200X80-10N" H 3200 2500 50  0001 C CNN
@@
 $EndComp
 $Comp
-L power:+3V3 #PWR048
+L power:+3V3 #PWR045
 U 1 1 5DE9BB40
 P 3850 1475
-F 0 "#PWR048" H 3850 1325 50  0001 C CNN
+F 0 "#PWR045" H 3850 1325 50  0001 C CNN
 F 1 "+3V3" H 3700 1550 50  0000 C CNN
 F 2 "" H 3850 1475 50  0001 C CNN
@@
 $EndComp
 $Comp
-L Device:C C19
+L Device:C C18
 U 1 1 5DE9BB48
 P 4175 1800
-F 0 "C19" V 3975 1800 50  0000 C CNN
+F 0 "C18" V 3975 1800 50  0000 C CNN
 F 1 "0.1u" V 4050 1800 50  0000 C CNN
 F 2 "Capacitor_SMD:C_0603_1608Metric" H 4213 1650 50  0001 C CNN
@@
 $EndComp
 $Comp
-L Device:C C18
+L Device:C C17
 U 1 1 5DE9BB50
 P 3625 1800
-F 0 "C18" V 3425 1800 50  0000 C CNN
+F 0 "C17" V 3425 1800 50  0000 C CNN
 F 1 "0.1u" V 3500 1800 50  0000 C CNN
 F 2 "Capacitor_SMD:C_0603_1608Metric" H 3663 1650 50  0001 C CNN
@@
 Connection ~ 3850 1800
 $Comp
-L power:+3V3 #PWR049
+L power:+3V3 #PWR046
 U 1 1 5DE9BB5C
 P 3950 1475
-F 0 "#PWR049" H 3950 1325 50  0001 C CNN
+F 0 "#PWR046" H 3950 1325 50  0001 C CNN
 F 1 "+3V3" H 4100 1550 50  0000 C CNN
 F 2 "" H 3950 1475 50  0001 C CNN
@@
 Connection ~ 3950 1800
 $Comp
-L power:GND #PWR050
+L power:GND #PWR047
 U 1 1 5DE9BB64
 P 3475 1800
-F 0 "#PWR050" H 3475 1550 50  0001 C CNN
+F 0 "#PWR047" H 3475 1550 50  0001 C CNN
 F 1 "GND" H 3480 1627 50  0000 C CNN
 F 2 "" H 3475 1800 50  0001 C CNN
@@
 $EndComp
 $Comp
-L power:GND #PWR051
+L power:GND #PWR048
 U 1 1 5DE9BB6A
 P 4325 1800
-F 0 "#PWR051" H 4325 1550 50  0001 C CNN
+F 0 "#PWR048" H 4325 1550 50  0001 C CNN
 F 1 "GND" H 4330 1627 50  0000 C CNN
 F 2 "" H 4325 1800 50  0001 C CNN
@@
 SDA
 $Comp
-L power:GND #PWR057
+L power:GND #PWR054
 U 1 1 5DE9BB73
 P 3900 3050
-F 0 "#PWR057" H 3900 2800 50  0001 C CNN
+F 0 "#PWR054" H 3900 2800 50  0001 C CNN
 F 1 "GND" H 3905 2877 50  0000 C CNN
 F 2 "" H 3900 3050 50  0001 C CNN
@@
 P 2825 2400
 AR Path="/5DE9BB83" Ref="R?"  Part="1"
-AR Path="/5DE92E14/5DE9BB83" Ref="R26"  Part="1"
-F 0 "R26" V 2725 2350 50  0000 L CNN
+AR Path="/5DE92E14/5DE9BB83" Ref="R25"  Part="1"
+F 0 "R25" V 2725 2350 50  0000 L CNN
 F 1 "NP" V 2825 2350 50  0000 L CNN
 F 2 "Resistor_SMD:R_0603_1608Metric" V 2755 2400 50  0001 C CNN
@@
 $EndComp
 $Comp
-L Device:R R29
+L Device:R R28
 U 1 1 5DE9BB8B
 P 2825 2800
-F 0 "R29" V 2725 2750 50  0000 L CNN
+F 0 "R28" V 2725 2750 50  0000 L CNN
 F 1 "10k" V 2825 2725 50  0000 L CNN
 F 2 "Resistor_SMD:R_0603_1608Metric" V 2755 2800 50  0001 C CNN
@@
 Connection ~ 2825 2600
 $Comp
-L power:GND #PWR056
+L power:GND #PWR053
 U 1 1 5DE9BB95
 P 2825 2950
-F 0 "#PWR056" H 2825 2700 50  0001 C CNN
+F 0 "#PWR053" H 2825 2700 50  0001 C CNN
 F 1 "GND" H 2830 2777 50  0000 C CNN
 F 2 "" H 2825 2950 50  0001 C CNN
@@
 $EndComp
 $Comp
-L power:+3V3 #PWR053
+L power:+3V3 #PWR050
 U 1 1 5DE9BB9B
 P 2825 2250
-F 0 "#PWR053" H 2825 2100 50  0001 C CNN
+F 0 "#PWR050" H 2825 2100 50  0001 C CNN
 F 1 "+3V3" H 2840 2423 50  0000 C CNN
 F 2 "" H 2825 2250 50  0001 C CNN
@@
 P 4725 2250
 AR Path="/5DE7F4ED" Ref="R?"  Part="1"
-AR Path="/5DE92E14/5DE7F4ED" Ref="R25"  Part="1"
-F 0 "R25" V 4625 2200 50  0000 L CNN
+AR Path="/5DE92E14/5DE7F4ED" Ref="R24"  Part="1"
+F 0 "R24" V 4625 2200 50  0000 L CNN
 F 1 "10k" V 4725 2175 50  0000 L CNN
 F 2 "Resistor_SMD:R_0603_1608Metric" V 4655 2250 50  0001 C CNN
@@
 $EndComp
 $Comp
-L power:+3V3 #PWR052
+L power:+3V3 #PWR049
 U 1 1 5DE7F4F3
 P 4725 2100
-F 0 "#PWR052" H 4725 1950 50  0001 C CNN
+F 0 "#PWR049" H 4725 1950 50  0001 C CNN
 F 1 "+3V3" H 4740 2273 50  0000 C CNN
 F 2 "" H 4725 2100 50  0001 C CNN
@@
 	4725 2400 4500 2400
 $Comp
-L resistors_0603:1-0000006 R27
+L resistors_0603:1-0000006 R26
 U 1 1 5FDB2113
 P 7825 2400
-F 0 "R27" V 7750 2400 50  0000 C CNN
+F 0 "R26" V 7750 2400 50  0000 C CNN
 F 1 "1-0000006" V 7825 2400 50  0001 C CNN
 F 2 "resistors_0603:1-0000006" V 7755 2400 50  0001 C CNN
@@
 $EndComp
 $Comp
-L resistors_0603:1-0000010 R28
+L resistors_0603:1-0000010 R27
 U 1 1 5FDB2B0F
 P 8050 2625
-F 0 "R28" V 8125 2575 50  0000 L CNN
+F 0 "R27" V 8125 2575 50  0000 L CNN
 F 1 "1-0000010" V 8050 2625 50  0001 C CNN
 F 2 "resistors_0603:1-0000010" V 7980 2625 50  0001 C CNN
@@
 $EndComp
 $Comp
-L power:GND #PWR054
+L power:GND #PWR051
 U 1 1 5FDB4AF1
 P 8425 2600
-F 0 "#PWR054" H 8425 2350 50  0001 C CNN
+F 0 "#PWR051" H 8425 2350 50  0001 C CNN
 F 1 "GND" H 8425 2450 50  0000 C CNN
 F 2 "" H 8425 2600 50  0001 C CNN
@@
 	8050 2400 8125 2400
 $Comp
-L power:GND #PWR055
+L power:GND #PWR052
 U 1 1 5FDB62BA
 P 8050 2775
-F 0 "#PWR055" H 8050 2525 50  0001 C CNN
+F 0 "#PWR052" H 8050 2525 50  0001 C CNN
 F 1 "GND" H 8050 2625 50  0000 C CNN
 F 2 "" H 8050 2775 50  0001 C CNN
@@
 Required mating block\n1-0000797
 $Comp
-L Connector_Generic:Conn_01x02 J5
+L Connector_Generic:Conn_01x02 J4
 U 1 1 5FDB68FF
 P 8625 1925
-F 0 "J5" H 8705 1917 50  0000 L CNN
+F 0 "J4" H 8705 1917 50  0000 L CNN
 F 1 "Hot Wire" H 8705 1826 50  0000 L CNN
 F 2 "lib_fp:1-0000783" H 8625 1925 50  0001 C CNN
