File: Hardware/Cutdown_PCB/KiCAD_Project/cutdown/cutdown.sch (KiCad schematic (older format))
At the start: 55 parts

Commit message: Remove cutdown power pcb and update cutdown design
Parts:
- removed C? (x2): 10u, symbol Device:C
- removed C? (x2): 1-0000007, capacitors_0603:1-0000007, symbol capacitors_0603:1-0000007
- removed F?: Polyfuse, symbol Device:Polyfuse
- removed U?: MIC5219-3.3YM5, Package_TO_SOT_SMD:SOT-23-5, symbol Regulator_Linear:MIC5219-3.3YM5
- added C10, C11, C13: 1-0000075, capacitors_0805:1-0000075, symbol capacitors_0805:1-0000075
- added C12: 1-0000018, capacitors_0603:1-0000018, symbol capacitors_0603:1-0000018
- added D4: D_Schottky, Diode_SMD:D_SOD-123F, symbol Device:D_Schottky
- added D5: Yellow, LED_SMD:LED_0805_2012Metric, symbol Device:LED_ALT
- added FID1, FID2: Fiducial, Fiducial:Fiducial_1mm_Mask2mm, symbol Mechanical:Fiducial
- added J3: External Cutdown, lib_fp:JST_S2B-PH-SM4-TB(LF)(SN), symbol Connector_Generic:Conn_01x02
- added PCB1: barepcb, lib_fp:barepcb, symbol lib_sch:barepcb
- added R13: 1-0000174, resistors_0603:1-0000174, symbol resistors_0603:1-0000174
- added R14: 1-0000013, resistors_0603:1-0000013, symbol resistors_0603:1-0000013
- added R15: 1-0000010, resistors_0603:1-0000010, symbol resistors_0603:1-0000010
- added U2: SPX3819M5-L-3-3, Package_TO_SOT_SMD:SOT-23-5, symbol Regulator_Linear:SPX3819M5-L-3-3
- added U4: MCP73831, lib_fp:1-0000793, symbol lib_sch:MCP73831
- C1, C15, C16, C2, C3, C4, C5, C6, C7, C8, C9: renamed from C?; Populated (none) -> 1; Population 1 -> (none)
- C17: renamed from C?; Populated (none) -> 0; Population 0 -> (none)
- D1, D2, D3, D6, D7, D8: renamed from D?; footprint (none) -> LED_SMD:LED_0805_2012Metric
- J1: renamed from J?; footprint (none) -> lib_fp:MiniUSB; Internal Part Number (none) -> 1-0000034; Populated (none) -> 1
- J2: renamed from J?; value Battery LiPO 2S -> Battery LiPO 1S; footprint (none) -> lib_fp:JST_S2B-PH-SM4-TB(LF)(SN); Internal Part Number 0-0000000 -> 1-0000526; Populated 0 -> 1
- J4: renamed from J?; footprint (none) -> Connector_PinHeader_2.54mm:PinHeader_2x03_P2.54mm_Vertical; Internal Part Number (none) -> 0-0000000; Populated (none) -> 0
- R16: renamed from R2; footprint Resistor_SMD:R_0603_1608Metric_Pad1.05x0.95mm_HandSolder -> Resistor_SMD:R_0603_1608Metric
- R17: renamed from R4; footprint Resistor_SMD:R_0603_1608Metric_Pad1.05x0.95mm_HandSolder -> Resistor_SMD:R_0603_1608Metric
- R19: renamed from R5; footprint Resistor_SMD:R_0603_1608Metric_Pad1.05x0.95mm_HandSolder -> Resistor_SMD:R_0603_1608Metric
- R20: renamed from R7; footprint Resistor_SMD:R_0603_1608Metric_Pad1.05x0.95mm_HandSolder -> Resistor_SMD:R_0603_1608Metric
- R21: renamed from R8; footprint Resistor_SMD:R_0603_1608Metric_Pad1.05x0.95mm_HandSolder -> Resistor_SMD:R_0603_1608Metric
- SW1: renamed from SW?; footprint (none) -> lib_fp:SW_GF-123-0054
- U1: renamed from U?; Internal Part Number (none) -> 1-0000779; Populated (none) -> 1
- U3: renamed from U?; Internal Part Number (none) -> 1-0000566; Populated (none) -> 1
- U5: renamed from U?; footprint (none) -> lib_fp:XBee
- Y1: renamed from Y?; footprint (none) -> lib_fp:Resonator; Internal Part Number (none) -> 1-0000569; Populated (none) -> 1
- gave numbers to parts that had none: 18
Connections:
- net labels added: +5V, +BATT
- wire segments 121 -> 139
- no-connect marks 28 -> 30
Other:
- moved on the sheet: C14, C15, C16, C17, D7, D8, J2, R22, R23, R24, SW1, U5
