File: Hardware/Cutdown_PCB/KiCAD_Project/cutdown/cutdown.sch (KiCad schematic (older format))
At the start: 10 parts, among them J1 Nichrome Wire, U1 Particle

Commit message: Cutdown PCB Rev 1.0 Complete.
Parts:
- R1, R2, R4, R5, R6, R7: Populated 0 -> 1
Connections:
- wire segments 22 -> 20
Other:
- note added: "Socket Particle with Header #1-0000295"
Changed lines of the file:
@@
 $EndComp
-Wire Wire Line
-	5825 7150 5775 7150
-Wire Wire Line
-	5775 7150 5775 6950
-Wire Wire Line
-	5775 6950 5825 6950
 Wire Wire Line
 	5825 7050 5725 7050
@@
 Text GLabel 5450 3300 0    50   Output ~ 0
 PIEZO_ELEMENT
-Wire Wire Line
-	5675 6950 5775 6950
-Connection ~ 5775 6950
 $Comp
 L lib_sch:Particle U1
@@
 F 3 "~" H 3400 6875 50  0001 C CNN
 F 4 "1-0000010" H 3400 6875 50  0001 C CNN "Internal Part Number"
-F 5 "0" H 3400 6875 50  0001 C CNN "Populated"
+F 5 "1" H 3400 6875 50  0001 C CNN "Populated"
 	1    3400 6875
 	0    1    1    0
@@
 F 3 "~" H 3400 6975 50  0001 C CNN
 F 4 "1-0000010" H 3400 6975 50  0001 C CNN "Internal Part Number"
-F 5 "0" H 3400 6975 50  0001 C CNN "Populated"
+F 5 "1" H 3400 6975 50  0001 C CNN "Populated"
 	1    3400 6975
 	0    1    1    0
@@
 F 3 "~" H 3400 7075 50  0001 C CNN
 F 4 "1-0000010" H 3400 7075 50  0001 C CNN "Internal Part Number"
-F 5 "0" H 3400 7075 50  0001 C CNN "Populated"
+F 5 "1" H 3400 7075 50  0001 C CNN "Populated"
 	1    3400 7075
 	0    1    1    0
@@
 F 3 "~" H 3400 7175 50  0001 C CNN
 F 4 "1-0000010" H 3400 7175 50  0001 C CNN "Internal Part Number"
-F 5 "0" H 3400 7175 50  0001 C CNN "Populated"
+F 5 "1" H 3400 7175 50  0001 C CNN "Populated"
 	1    3400 7175
 	0    1    1    0
@@
 F 3 "~" H 3400 7275 50  0001 C CNN
 F 4 "1-0000010" H 3400 7275 50  0001 C CNN "Internal Part Number"
-F 5 "0" H 3400 7275 50  0001 C CNN "Populated"
+F 5 "1" H 3400 7275 50  0001 C CNN "Populated"
 	1    3400 7275
 	0    1    1    0
@@
 F 3 "~" H 3400 7375 50  0001 C CNN
 F 4 "1-0000010" H 3400 7375 50  0001 C CNN "Internal Part Number"
-F 5 "0" H 3400 7375 50  0001 C CNN "Populated"
+F 5 "1" H 3400 7375 50  0001 C CNN "Populated"
 	1    3400 7375
 	0    1    1    0
@@
 Wire Wire Line
 	3675 7475 3675 7525
+Text GLabel 5375 7150 0    50   Input ~ 0
+EXT_CUTDOWN
+Wire Wire Line
+	5675 6950 5825 6950
+Wire Wire Line
+	5375 7150 5825 7150
+Text Notes 5300 2250 0    50   ~ 0
+Socket Particle with Header #1-0000295
 $EndSCHEMATC

Commit message: Fix GPS connection to particle.
Parts:
- added R14, R15: 0R0, Resistor_SMD:R_0603_1608Metric_Pad1.05x0.95mm_HandSolder, symbol Device:R
- R1, R2, R3, R4, R5, R6, R7, R8: footprint Resistors_SMD:R_0603_HandSoldering -> Resistor_SMD:R_0603_1608Metric_Pad1.05x0.95mm_HandSolder
Connections:
- wire segments 20 -> 22
Changed lines of the file:
@@
 EESchema Schematic File Version 4
-LIBS:cutdown-cache
 EELAYER 30 0
 EELAYER END
@@
 Sheet 1 2
 Title "Cutdown Module - NSSL EFM"
-Date "2019-12-03"
-Rev "1.0"
+Date "2020-03-30"
+Rev "2.0"
 Comp "Leeman Geophysical LLC"
 Comment1 "(479) 373-3736"
@@
 F 0 "R3" V 5450 6950 50  0000 C CNN
 F 1 "0R0" V 5525 6950 50  0000 C CNN
-F 2 "Resistors_SMD:R_0603_HandSoldering" V 5455 6950 50  0001 C CNN
+F 2 "Resistor_SMD:R_0603_1608Metric_Pad1.05x0.95mm_HandSolder" V 5455 6950 50  0001 C CNN
 F 3 "~" H 5525 6950 50  0001 C CNN
 F 4 "1-0000006" H 5525 6950 50  0001 C CNN "Internal Part Number"
@@
 Text GLabel 6850 3500 2    50   Input ~ 0
 BMP388_INT
-Text GLabel 6850 3600 2    50   Input ~ 0
+Text GLabel 5050 4100 0    50   Input ~ 0
 GPS_RX
-Text GLabel 6850 3700 2    50   Output ~ 0
+Text GLabel 5050 4000 0    50   Output ~ 0
 GPS_TX
 $Comp
@@
 NoConn ~ 6850 4100
 NoConn ~ 6850 4200
-NoConn ~ 5450 4100
-NoConn ~ 5450 4000
 NoConn ~ 5450 3400
 NoConn ~ 5450 3500
@@
 F 0 "R1" V 3350 7000 50  0000 L CNN
 F 1 "10k" V 3400 6800 50  0000 L CNN
-F 2 "Resistors_SMD:R_0603_HandSoldering" V 3330 6875 50  0001 C CNN
+F 2 "Resistor_SMD:R_0603_1608Metric_Pad1.05x0.95mm_HandSolder" V 3330 6875 50  0001 C CNN
 F 3 "~" H 3400 6875 50  0001 C CNN
 F 4 "1-0000010" H 3400 6875 50  0001 C CNN "Internal Part Number"
@@
 F 0 "R2" V 3350 7100 50  0000 L CNN
 F 1 "10k" V 3400 6900 50  0000 L CNN
-F 2 "Resistors_SMD:R_0603_HandSoldering" V 3330 6975 50  0001 C CNN
+F 2 "Resistor_SMD:R_0603_1608Metric_Pad1.05x0.95mm_HandSolder" V 3330 6975 50  0001 C CNN
 F 3 "~" H 3400 6975 50  0001 C CNN
 F 4 "1-0000010" H 3400 6975 50  0001 C CNN "Internal Part Number"
@@
 F 0 "R4" V 3350 7200 50  0000 L CNN
 F 1 "10k" V 3400 7000 50  0000 L CNN
-F 2 "Resistors_SMD:R_0603_HandSoldering" V 3330 7075 50  0001 C CNN
+F 2 "Resistor_SMD:R_0603_1608Metric_Pad1.05x0.95mm_HandSolder" V 3330 7075 50  0001 C CNN
 F 3 "~" H 3400 7075 50  0001 C CNN
 F 4 "1-0000010" H 3400 7075 50  0001 C CNN "Internal Part Number"
@@
 F 0 "R5" V 3350 7300 50  0000 L CNN
 F 1 "10k" V 3400 7100 50  0000 L CNN
-F 2 "Resistors_SMD:R_0603_HandSoldering" V 3330 7175 50  0001 C CNN
+F 2 "Resistor_SMD:R_0603_1608Metric_Pad1.05x0.95mm_HandSolder" V 3330 7175 50  0001 C CNN
 F 3 "~" H 3400 7175 50  0001 C CNN
 F 4 "1-0000010" H 3400 7175 50  0001 C CNN "Internal Part Number"
@@
 F 0 "R6" V 3350 7400 50  0000 L CNN
 F 1 "10k" V 3400 7200 50  0000 L CNN
-F 2 "Resistors_SMD:R_0603_HandSoldering" V 3330 7275 50  0001 C CNN
+F 2 "Resistor_SMD:R_0603_1608Metric_Pad1.05x0.95mm_HandSolder" V 3330 7275 50  0001 C CNN
 F 3 "~" H 3400 7275 50  0001 C CNN
 F 4 "1-0000010" H 3400 7275 50  0001 C CNN "Internal Part Number"
@@
 F 0 "R7" V 3350 7500 50  0000 L CNN
 F 1 "10k" V 3400 7300 50  0000 L CNN
-F 2 "Resistors_SMD:R_0603_HandSoldering" V 3330 7375 50  0001 C CNN
+F 2 "Resistor_SMD:R_0603_1608Metric_Pad1.05x0.95mm_HandSolder" V 3330 7375 50  0001 C CNN
 F 3 "~" H 3400 7375 50  0001 C CNN
 F 4 "1-0000010" H 3400 7375 50  0001 C CNN "Internal Part Number"
@@
 F 0 "R8" V 3350 7600 50  0000 L CNN
 F 1 "NP" V 3400 7425 50  0000 L CNN
-F 2 "Resistors_SMD:R_0603_HandSoldering" V 3330 7475 50  0001 C CNN
+F 2 "Resistor_SMD:R_0603_1608Metric_Pad1.05x0.95mm_HandSolder" V 3330 7475 50  0001 C CNN
 F 3 "~" H 3400 7475 50  0001 C CNN
 F 4 "1-0000010" H 3400 7475 50  0001 C CNN "Internal Part Number"
@@
 Text Notes 5300 2250 0    50   ~ 0
 Socket Particle with Header #1-0000295
+$Comp
+L Device:R R14
+U 1 1 5E82303F
+P 5300 4000
+F 0 "R14" V 5225 3825 50  0000 C CNN
+F 1 "0R0" V 5300 4000 50  0000 C CNN
+F 2 "Resistor_SMD:R_0603_1608Metric_Pad1.05x0.95mm_HandSolder" V 5230 4000 50  0001 C CNN
+F 3 "~" H 5300 4000 50  0001 C CNN
+F 4 "1-0000006" H 5300 4000 50  0001 C CNN "Internal Part Number"
+F 5 "1" H 5300 4000 50  0001 C CNN "Populated"
+	1    5300 4000
+	0    1    1    0
+$EndComp
+$Comp
+L Device:R R15
+U 1 1 5E823B07
+P 5300 4100
+F 0 "R15" V 5250 3925 50  0000 C CNN
+F 1 "0R0" V 5300 4100 50  0000 C CNN
+F 2 "Resistor_SMD:R_0603_1608Metric_Pad1.05x0.95mm_HandSolder" V 5230 4100 50  0001 C CNN
+F 3 "~" H 5300 4100 50  0001 C CNN
+F 4 "1-0000006" H 5300 4100 50  0001 C CNN "Internal Part Number"
+F 5 "1" H 5300 4100 50  0001 C CNN "Populated"
+	1    5300 4100
+	0    1    1    0
+$EndComp
+Wire Wire Line
+	5150 4000 5050 4000
+Wire Wire Line
+	5050 4100 5150 4100
+NoConn ~ 6850 3600
+NoConn ~ 6850 3700
 $EndSCHEMATC

Commit message: Rework cutdown schematic for version 2
Parts:
- removed J1: Nichrome Wire, Pin_Headers:Pin_Header_Straight_1x04_Pitch2.54mm, symbol Connector_Generic:Conn_01x04
- removed R1, R6: 10k, Resistor_SMD:R_0603_1608Metric_Pad1.05x0.95mm_HandSolder, symbol Device:R
- removed R14, R15, R3: 0R0, Resistor_SMD:R_0603_1608Metric_Pad1.05x0.95mm_HandSolder, symbol Device:R
- removed U1: Particle, lib_fp:Particle, symbol lib_sch:Particle
- added C? (x11): 1-0000007, capacitors_0603:1-0000007, symbol capacitors_0603:1-0000007
- added C?: 1-0000075, capacitors_0805:1-0000075, symbol capacitors_0805:1-0000075
- added C?: 1-0000018, capacitors_0603:1-0000018, symbol capacitors_0603:1-0000018
- added C? (x2): 1-0000017, capacitors_0603:1-0000017, symbol capacitors_0603:1-0000017
- added C? (x2): 10u, symbol Device:C
- added D?: Green, symbol Device:LED_ALT
- added D? (x2): Red, symbol Device:LED_ALT
- added D? (x2): Yellow, symbol Device:LED_ALT
- added D?: Blue, symbol Device:LED_ALT
- added F?: Polyfuse, symbol Device:Polyfuse
- added J?: ISP, symbol Connector_Generic:Conn_02x03_Counter_Clockwise
- added J?: Mini_USB_B, symbol lib_sch:Mini_USB_B
- added J?: Battery LiPO 2S, symbol Connector_Generic:Conn_01x02
- added Q?: 2N7002, Package_TO_SOT_SMD:SOT-23, symbol Transistor_FET:2N7002
- added R? (x6): 1-0000008, resistors_0603:1-0000008, symbol resistors_0603:1-0000008
- added R? (x3): 1-0000006, resistors_0603:1-0000006, symbol resistors_0603:1-0000006
- added R? (x3): 1-0000010, resistors_0603:1-0000010, symbol resistors_0603:1-0000010
- added R? (x2): 1-0000013, resistors_0603:1-0000013, symbol resistors_0603:1-0000013
- added R? (x2): 1-0000012, resistors_0603:1-0000012, symbol resistors_0603:1-0000012
- added SW?: SW_SPST, symbol Switch:SW_SPST
- added U?: ATmega328P-AU, Package_QFP:TQFP-32_7x7mm_P0.8mm, symbol lib_sch:ATmega328P-AU
- added U?: XBee, symbol lib_sch:XBee
- added U?: FT231XS, Package_SO:SSOP-20_3.9x8.7mm_P0.635mm, symbol Interface_USB:FT231XS
- added U?: MIC5219-3.3YM5, Package_TO_SOT_SMD:SOT-23-5, symbol Regulator_Linear:MIC5219-3.3YM5
- added Y?: 16MHz, symbol Device:Resonator_Small
Connections:
- net labels added: Cutdown_Command, DTR, MISO, MOSI, RESET, RXI, SCK, TXO, XBee_from_uC, XBee_to_uC
- net labels removed: BMP388_SDO, CUTOFF_LOGIC, GPS_PPS, GPS_RX, GPS_TX, PIEZO_ELEMENT
- wire segments 22 -> 121
- no-connect marks 15 -> 28
Other:
- note added: "Power Indicator"
- note removed: "Socket Particle with Header #1-0000295"
- moved on the sheet: R2, R4, R5, R7, R8

Commit message: Initial layout
Parts:
- removed C? (x2): 10u, symbol Device:C
- removed C? (x2): 1-0000007, capacitors_0603:1-0000007, symbol capacitors_0603:1-0000007
- removed F?: Polyfuse, symbol Device:Polyfuse
- removed U?: MIC5219-3.3YM5, Package_TO_SOT_SMD:SOT-23-5, symbol Regulator_Linear:MIC5219-3.3YM5
- added C10, C11, C13: 1-0000075, capacitors_0805:1-0000075, symbol capacitors_0805:1-0000075
- added C12: 1-0000018, capacitors_0603:1-0000018, symbol capacitors_0603:1-0000018
- added D7: D_Schottky, Diode_SMD:D_SOD-123F, symbol Device:D_Schottky
- added D8: Yellow, LED_SMD:LED_0805_2012Metric, symbol Device:LED_ALT
- added J5: External Cutdown, lib_fp:JST_S2B-PH-SM4-TB(LF)(SN), symbol Connector_Generic:Conn_01x02
- added PCB1: barepcb, lib_fp:barepcb, symbol lib_sch:barepcb
- added R27: 1-0000174, resistors_0603:1-0000174, symbol resistors_0603:1-0000174
- added R28: 1-0000013, resistors_0603:1-0000013, symbol resistors_0603:1-0000013
- added R29: 1-0000010, resistors_0603:1-0000010, symbol resistors_0603:1-0000010
- added U2: SPX3819M5-L-3-3, Package_TO_SOT_SMD:SOT-23-5, symbol Regulator_Linear:SPX3819M5-L-3-3
- added U6: MCP73831, lib_fp:1-0000793, symbol lib_sch:MCP73831
- D1, D2, D3, D4, D5, D6: renamed from D?; footprint (none) -> LED_SMD:LED_0805_2012Metric
- J1: renamed from J?; footprint (none) -> lib_fp:MiniUSB
- J2: renamed from J?; value Battery LiPO 2S -> Battery LiPO 1S; footprint (none) -> lib_fp:JST_S2B-PH-SM4-TB(LF)(SN); Internal Part Number 0-0000000 -> 1-0000526; Populated 0 -> 1
- J3: renamed from J?; footprint (none) -> Connector_PinHeader_2.54mm:PinHeader_2x03_P2.54mm_Vertical
- R13: renamed from R2; footprint Resistor_SMD:R_0603_1608Metric_Pad1.05x0.95mm_HandSolder -> Resistor_SMD:R_0603_1608Metric
- R14: renamed from R4; footprint Resistor_SMD:R_0603_1608Metric_Pad1.05x0.95mm_HandSolder -> Resistor_SMD:R_0603_1608Metric
- R16: renamed from R5; footprint Resistor_SMD:R_0603_1608Metric_Pad1.05x0.95mm_HandSolder -> Resistor_SMD:R_0603_1608Metric
- R17: renamed from R7; footprint Resistor_SMD:R_0603_1608Metric_Pad1.05x0.95mm_HandSolder -> Resistor_SMD:R_0603_1608Metric
- R18: renamed from R8; footprint Resistor_SMD:R_0603_1608Metric_Pad1.05x0.95mm_HandSolder -> Resistor_SMD:R_0603_1608Metric
- SW1: renamed from SW?; footprint (none) -> lib_fp:SW_GF-123-0054
- U4: renamed from U?; footprint (none) -> lib_fp:XBee
- Y1: renamed from Y?; footprint (none) -> lib_fp:Resonator
- gave numbers to parts that had none: 32
Connections:
- net labels added: +5V, +BATT
- wire segments 121 -> 139
- no-connect marks 28 -> 27
Other:
- note added: "CHECK POLARITY"
- moved on the sheet: C14, C15, C16, C17, D5, D6, J2, R19, R20, R21, SW1, U4

Commit message: Tweak schematic and PCB
Parts:
- added FID1, FID2: Fiducial, Fiducial:Fiducial_1mm_Mask2mm, symbol Mechanical:Fiducial
- C1, C12, C15, C16, C2, C3, C4, C5, C6, C7, C8, C9: Populated (none) -> 1; Population 1 -> (none)
- C17: Populated (none) -> 0; Population 0 -> (none)
- J1: Internal Part Number (none) -> 1-0000034; Populated (none) -> 1
- J3: renamed from J5; Internal Part Number (none) -> 1-0000526; Populated (none) -> 1
- J4: renamed from J3; Internal Part Number (none) -> 0-0000000; Populated (none) -> 0
- U1: Internal Part Number (none) -> 1-0000779; Populated (none) -> 1
- U3: Internal Part Number (none) -> 1-0000566; Populated (none) -> 1
- U4: renamed from U6; Internal Part Number (none) -> 1-0000793; Populated (none) -> 1
- Y1: Internal Part Number (none) -> 1-0000569; Populated (none) -> 1
- renumbered D7 to D4, D8 to D5, D4 to D6, D5 to D7, D6 to D8, R27 to R13, R28 to R14, R29 to R15, R13 to R16, R14 to R17, R15 to R18, R16 to R19, R17 to R20, R18 to R21, R19 to R22, R20 to R23, R21 to R24, U4 to U5
Connections:
- no-connect marks 27 -> 30
Other:
- note removed: "CHECK POLARITY"

Commit message: Cutdown hardware updates
Parts:
- R7, R8: Internal Part Number 1-0000006 -> 1-0000012
- Y1: value 16MHz -> 8MHz; Internal Part Number 1-0000569 -> 1-0000721
Other:
- note added: "Ext Cutdown Cable 1-0000804"
- note added: "Li-Ion Battery Options:\n350mAh 1-0000807\n150mAh 1-0000806\n105 mAh 1-0000805\n"
- note added: "Optional Socket for XBee 1-0000050"
Changed lines of the file:
@@
 P 8825 3675
 F 0 "Y1" V 8520 3625 50  0000 C CNN
-F 1 "16MHz" V 8611 3625 50  0000 C CNN
+F 1 "8MHz" V 8611 3625 50  0000 C CNN
 F 2 "lib_fp:Resonator" H 8800 3675 50  0001 C CNN
 F 3 "~" H 8800 3675 50  0001 C CNN
-F 4 "1-0000569" H 8825 3675 50  0001 C CNN "Internal Part Number"
+F 4 "1-0000721" H 8825 3675 50  0001 C CNN "Internal Part Number"
 F 5 "1" H 8825 3675 50  0001 C CNN "Populated"
 	1    8825 3675
@@
 Text GLabel 10225 5025 2    50   Output ~ 0
 XBee_from_uC
-$Comp
-L lib_sch:XBee U5
-U 1 1 5FDD2C3A
-P 3775 7050
-F 0 "U5" H 3775 7747 60  0000 C CNN
-F 1 "XBee" H 3775 7641 60  0000 C CNN
-F 2 "lib_fp:XBee" H 3800 7050 60  0001 C CNN
-F 3 "" H 3800 7050 60  0001 C CNN
-F 4 "1-0000785" H 3775 7050 50  0001 C CNN "Internal Part Number"
-F 5 "1" H 3775 7050 50  0001 C CNN "Populated"
-	1    3775 7050
-	1    0    0    -1
-$EndComp
 $Comp
 L capacitors_0805:1-0000075 C14
@@
 F 2 "resistors_0603:1-0000012" V 2655 1650 50  0001 C CNN
 F 3 "~" H 2725 1650 50  0001 C CNN
-F 4 "1-0000006" H 2725 1650 50  0001 C CNN "Internal Part Number"
+F 4 "1-0000012" H 2725 1650 50  0001 C CNN "Internal Part Number"
 F 5 "1" H 2725 1650 50  0001 C CNN "Populated"
 F 6 "27" V 2725 1650 50  0000 C CNN "PValue"
@@
 F 2 "resistors_0603:1-0000012" V 2655 1750 50  0001 C CNN
 F 3 "~" H 2725 1750 50  0001 C CNN
-F 4 "1-0000006" H 2725 1750 50  0001 C CNN "Internal Part Number"
+F 4 "1-0000012" H 2725 1750 50  0001 C CNN "Internal Part Number"
 F 5 "1" H 2725 1750 50  0001 C CNN "Populated"
 F 6 "27" V 2725 1750 50  0000 C CNN "PValue"
@@
 	1    0    0    -1
 $EndComp
+Text Notes 3075 7650 0    50   ~ 0
+Optional Socket for XBee 1-0000050
+$Comp
+L lib_sch:XBee U5
+U 1 1 5FDD2C3A
+P 3775 7050
+F 0 "U5" H 3775 7747 60  0000 C CNN
+F 1 "XBee" H 3775 7641 60  0000 C CNN
+F 2 "lib_fp:XBee" H 3800 7050 60  0001 C CNN
+F 3 "" H 3800 7050 60  0001 C CNN
+F 4 "1-0000785" H 3775 7050 50  0001 C CNN "Internal Part Number"
+F 5 "1" H 3775 7050 50  0001 C CNN "Populated"
+	1    3775 7050
+	1    0    0    -1
+$EndComp
+Text Notes 675  4075 0    50   ~ 0
+Li-Ion Battery Options:\n350mAh 1-0000807\n150mAh 1-0000806\n105 mAh 1-0000805\n
+Text Notes 6425 4100 0    50   ~ 0
+Ext Cutdown Cable 1-0000804
 $EndSCHEMATC
