File: Hardware/Digital_PCB/KiCAD_Project/digital_pcb/digital_pcb.sch (KiCad schematic (older format))
At the start: 36 parts, among them J1 Conn_01x02, J2 ISP, J3 Conn_01x02, J4 Spare 1, J5 Board to Board, U1 STM32F103CBTx, Y1 8MHz

Commit message: Digital PCB revs
Parts:
- PCB1: Internal Part Number 3-0000069 -> 3-0000129
Changed lines of the file:
@@
 Sheet 1 5
 Title "Digital Rotating Electronics - NSSL EFM"
-Date "2020-12-18"
-Rev "3.0"
+Date "2022-02-25"
+Rev "3.1"
 Comp "Leeman Geophysical LLC"
 Comment1 "(479) 373-3736"
@@
 F 2 "lib_fp:barepcb" H 7225 6400 50  0001 C CNN
 F 3 "" H 7225 6400 50  0001 C CNN
-F 4 "3-0000069" H 7225 6400 50  0001 C CNN "Internal Part Number"
+F 4 "3-0000129" H 7225 6400 50  0001 C CNN "Internal Part Number"
 F 5 "1" H 7225 6400 50  0001 C CNN "Populated"
 	1    7225 6400
